File: cad/watch_pcb/watch_pcb.kicad_pcb (KiCad board)
At the start: 2 copper layers, 34 x 40 mm, 16 parts, among them J1 DISPLAY, J4 USB_C_Receptacle, U1 LIS3MDL, U10 MX25LM51245GXDI00, U11 LSM6DSV16XTR, U2 MAX-M10M, U3 AMS1117-3.3, U4 FT231XQ, U5 AP131-18, U6 MAX30102, U7 MCP73871-2AA, U8 ESP32-S3, U9 S80KS5123GABHI020

Commit message: more
Parts:
- removed U4: FT231XQ, Package_DFN_QFN:QFN-20-1EP_4x4mm_P0.5mm_EP2.5x2.5mm
- added C1: 22uF, Capacitor_SMD:C_0603_1608Metric, F.Cu at (120.0, 98.0)
- added C10: 100nF, Capacitor_SMD:C_0201_0603Metric, F.Cu at (149.7, 89.5)
- added C11: 100nF, Capacitor_SMD:C_0201_0603Metric, F.Cu at (149.7, 91.4)
- added C12: 1uF, Capacitor_SMD:C_0402_1005Metric, F.Cu at (137.8, 91.3)
- added C13: 10uF, Capacitor_SMD:C_0402_1005Metric, B.Cu at (101.2, 84.6)
- added C14: 10nF, Capacitor_SMD:C_0201_0603Metric, B.Cu at (104.0, 102.0)
- added C15: 100nF, Capacitor_SMD:C_0201_0603Metric, F.Cu at (128.6, 106.5)
- added C18: 10uF, Capacitor_SMD:C_0402_1005Metric, F.Cu at (137.8, 96.4)
- added C19: 4.7uF, Capacitor_SMD:C_0603_1608Metric, F.Cu at (146.0, 93.1)
- added C2: 22uF, Capacitor_SMD:C_0603_1608Metric, F.Cu at (122.0, 105.6)
- added C20: 4.7uF, Capacitor_SMD:C_0603_1608Metric, F.Cu at (146.0, 96.1)
- added C25: 1uF, Capacitor_SMD:C_0402_1005Metric, F.Cu at (141.8, 83.8)
- added C26: 10nF, Capacitor_SMD:C_0201_0603Metric, F.Cu at (152.5, 85.5)
- added C27: 100nF, Capacitor_SMD:C_0201_0603Metric, F.Cu at (152.5, 87.5)
- added C28: 1uF, Capacitor_SMD:C_0402_1005Metric, F.Cu at (141.8, 86.3)
- added C29: 1uF, Capacitor_SMD:C_0402_1005Metric, F.Cu at (141.8, 88.8)
- added C3: 1uF, Capacitor_SMD:C_0402_1005Metric, F.Cu at (128.4, 100.2)
- added C30: 100nF, Capacitor_SMD:C_0201_0603Metric, F.Cu at (152.5, 89.5)
- added C31: 100nF, Capacitor_SMD:C_0201_0603Metric, F.Cu at (152.5, 91.4)
- added C32: 100nF, Capacitor_SMD:C_0201_0603Metric, F.Cu at (152.5, 93.4)
- added C33: 100nF, Capacitor_SMD:C_0201_0603Metric, F.Cu at (155.4, 83.5)
- added C34: 1uF, Capacitor_SMD:C_0402_1005Metric, F.Cu at (141.8, 91.3)
- added C35: 10uF, Capacitor_SMD:C_0402_1005Metric, F.Cu at (141.8, 93.9)
- added C36: 100nF, Capacitor_SMD:C_0201_0603Metric, F.Cu at (155.4, 85.5)
- added C37: 100nF, Capacitor_SMD:C_0201_0603Metric, F.Cu at (155.4, 87.5)
- added C4: 100nF, Capacitor_SMD:C_0201_0603Metric, F.Cu at (132.8, 103.2)
- added C5: 10uF, Capacitor_SMD:C_0402_1005Metric, F.Cu at (131.9, 98.2)
- added C6: 10uF, Capacitor_SMD:C_0402_1005Metric, F.Cu at (137.8, 88.8)
- added C7: 100nF, Capacitor_SMD:C_0201_0603Metric, F.Cu at (149.7, 85.5)
- added C8: 100nF, Capacitor_SMD:C_0201_0603Metric, F.Cu at (149.7, 87.5)
- added C9: 4.7uF, Capacitor_SMD:C_0603_1608Metric, F.Cu at (146.0, 90.1)
- added J2: Micro_SD_Card, 5033981892:MOLEX_503398-1892, F.Cu at (108.2, 86.8)
- added R1: 5.1k, Resistor_SMD:R_0402_1005Metric, F.Cu at (156.8, 96.7)
- added R11: 100k, Resistor_SMD:R_0402_1005Metric, B.Cu at (131.8, 106.4)
- added R12: 2k, Resistor_SMD:R_0402_1005Metric, F.Cu at (159.8, 102.6)
- added R13: 50k, Resistor_SMD:R_0402_1005Metric, F.Cu at (159.8, 104.6)
- added R14: 470, Resistor_SMD:R_0402_1005Metric, F.Cu at (159.8, 106.6)
- added R15: 1k, Resistor_SMD:R_0402_1005Metric, F.Cu at (159.8, 108.6)
- added R16: 1k, Resistor_SMD:R_0402_1005Metric, F.Cu at (162.7, 96.7)
- added R18: 10k, Resistor_SMD:R_0402_1005Metric, F.Cu at (162.7, 98.7)
- added R19: 10k, Resistor_SMD:R_0402_1005Metric, F.Cu at (162.7, 100.6)
- added R2: 5.1k, Resistor_SMD:R_0402_1005Metric, F.Cu at (156.8, 98.7)
- added R20: 10k, Resistor_SMD:R_0402_1005Metric, F.Cu at (162.7, 102.6)
- added R21: 0, Resistor_SMD:R_0402_1005Metric, F.Cu at (125.6, 61.6)
- added R22: 0, Resistor_SMD:R_0402_1005Metric, F.Cu at (125.6, 63.6)
- added R23: 0, Resistor_SMD:R_0402_1005Metric, F.Cu at (128.0, 80.2)
- added R24: 0, Resistor_SMD:R_0402_1005Metric, F.Cu at (128.5, 53.6)
- added R25: 0, Resistor_SMD:R_0402_1005Metric, F.Cu at (128.5, 55.6)
- added R26: 0, Resistor_SMD:R_0402_1005Metric, F.Cu at (128.5, 57.6)
- added R27: 0, Resistor_SMD:R_0402_1005Metric, F.Cu at (128.5, 59.6)
- added R28: 0, Resistor_SMD:R_0402_1005Metric, F.Cu at (128.5, 61.6)
- added R29: 0, Resistor_SMD:R_0402_1005Metric, F.Cu at (128.5, 63.6)
- added R3: 1k, Resistor_SMD:R_0402_1005Metric, F.Cu at (156.8, 100.6)
- added R30: 0, Resistor_SMD:R_0402_1005Metric, B.Cu at (122.0, 81.6)
- added R31: 10k, Resistor_SMD:R_0402_1005Metric, F.Cu at (168.5, 96.7)
- added R32: 10k, Resistor_SMD:R_0402_1005Metric, B.Cu at (104.2, 90.2)
- added R33: 2k, Resistor_SMD:R_0402_1005Metric, F.Cu at (168.5, 100.6)
- added R34: 2k, Resistor_SMD:R_0402_1005Metric, F.Cu at (168.5, 102.6)
- added R35: R, Resistor_SMD:R_0402_1005Metric, F.Cu at (168.5, 104.6)
- added R36: R, Resistor_SMD:R_0402_1005Metric, F.Cu at (168.5, 106.6)
- added R4: 10k, Resistor_SMD:R_0402_1005Metric, B.Cu at (103.7, 82.6)
- added R5: 10k, Resistor_SMD:R_0402_1005Metric, B.Cu at (105.0, 85.4)
- added R6: 10k, Resistor_SMD:R_0402_1005Metric, B.Cu at (104.6, 80.9)
- added R7: 10k, Resistor_SMD:R_0402_1005Metric, B.Cu at (103.8, 86.6)
- added R8: 10k, Resistor_SMD:R_0402_1005Metric, B.Cu at (101.2, 87.6)
- added R9: 10k, Resistor_SMD:R_0402_1005Metric, F.Cu at (159.8, 98.7)
- added TP1: BOOT, TestPoint:TestPoint_Pad_D2.0mm, B.Cu at (90.0, 87.4)
- added TP2: GND, TestPoint:TestPoint_Pad_2.0x2.0mm, B.Cu at (86.0, 87.4)
- added TP3: BATT-, TestPoint:TestPoint_Pad_2.5x2.5mm, F.Cu at (125.4, 105.6)
- added TP4: BATT+, TestPoint:TestPoint_Pad_D2.5mm, F.Cu at (125.4, 100.8)
- D3, U1, U10, U9: moved to B.Cu
- J4: footprint Inset USB-C:CU3024PAAHLR001-NH_CVI -> DX07B024JJ1R1500:JAE_DX07B024JJ1R1500
- moved U1 41.2 mm to (103.2, 76.6), turned to 180 degrees
- moved D3 28.1 mm to (104.0, 100.8), turned to 180 degrees
- moved J4 22.2 mm to (107.2, 101.2)
- moved U5 18.9 mm to (131.4, 100.6), turned to 0 degrees
- moved U10 16.1 mm to (113.2, 77.4), turned to -90 degrees
- moved U9 13.0 mm to (127.2, 77.4), turned to 90 degrees
- moved U2 11.7 mm to (127.6, 91.5), turned to 90 degrees
- moved U3 10.8 mm to (116.2, 103.4), turned to 180 degrees
- moved U7 7.67 mm to (114.1, 96.8), turned to 180 degrees
- moved U8 7.18 mm to (120.4, 79.2), turned to -90 degrees
- moved MK1 4.54 mm to (132.3, 105.8)
- moved U11 0.87 mm to (117.6, 88.4), turned to 90 degrees
- moved U6 0.80 mm to (117.4, 88.4)
Connections:
- net Net-(J3-Pin_1) renamed /BATT+
- U1 pad 1: unconnected-(U1-SCL/SPC-Pad1) -> /IMU_SCL
- U1 pad 11: unconnected-(U1-SDA/SDI/SDO-Pad11) -> /IMU_SDA
- U11 pad 1: unconnected-(U11-SDO/SA0-Pad1) -> GND
- U11 pad 12: unconnected-(U11-CS-Pad12) -> +3V3
- U11 pad 13: unconnected-(U11-SCL-Pad13) -> /I2C1_SCL
- U11 pad 14: unconnected-(U11-SDA-Pad14) -> /I2C1_SDA
- U11 pad 2: unconnected-(U11-SDx/AH1/QVAR1-Pad2) -> /IMU_SDA
- U11 pad 3: unconnected-(U11-SCx/AH2/QVAR2-Pad3) -> /IMU_SCL
- U8 pad 10: /SPI3_ -> unconnected-(U8-GPIO5-Pad10)
- U8 pad 11: /SPI3_ -> unconnected-(U8-GPIO6-Pad11)
- U8 pad 12: /SPI3_ -> unconnected-(U8-GPIO7-Pad12)
- U8 pad 49: Net-(U8-U0TXD) -> unconnected-(U8-U0TXD-Pad49)
- U8 pad 5: unconnected-(U8-GPIO0-Pad5) -> /I2C1_SCL
- U8 pad 50: /UART_MOSI -> unconnected-(U8-U0RXD-Pad50)
- U8 pad 52: unconnected-(U8-GPIO46-Pad52) -> Net-(U8-GPIO46)
- U8 pad 6: unconnected-(U8-GPIO1-Pad6) -> /I2C1_SDA
- U8 pad 7: /I2C1_SCL -> unconnected-(U8-GPIO2-Pad7)
- U8 pad 8: /I2C1_SDA -> unconnected-(U8-GPIO3-Pad8)
- U8 pad 9: /SPI3_ -> unconnected-(U8-GPIO4-Pad9)
Routing:
- added copper zone on B.Cu, net GND
- added copper zone on F.Cu, net GND
- added copper zone on In1.Cu, net GND
- added copper zone on In2.Cu, net GND
Other:
- outline, holes or cut-outs redrawn
- copper layers 2 -> 4
- board text removed: "write stuff here!!"

Commit message: idk some stuff
Parts:
- removed AE1: Antenna_Dipole, RF_Antenna:Texas_SWRA117D_2.4GHz_Right
- removed C1, C2: 22uF, Capacitor_SMD:C_0603_1608Metric
- removed J1: DISPLAY, Connector_FFC-FPC:Hirose_FH12-18S-0.5SH_1x18-1MP_P0.50mm_Horizontal
- removed TP1: BOOT, TestPoint:TestPoint_Pad_D2.0mm
- removed TP2: GND, TestPoint:TestPoint_Pad_2.0x2.0mm
- removed U3: AMS1117-3.3, Package_TO_SOT_SMD:SOT-223-3_TabPin2
- added C16: 100nF, Capacitor_SMD:C_0201_0603Metric, F.Cu at (176.6, 108.0)
- added C17: 1uF, Capacitor_SMD:C_0402_1005Metric, F.Cu at (158.3, 99.0)
- added C21: C, Capacitor_SMD:C_0402_1005Metric, F.Cu at (158.3, 102.9)
- added C22: 1.5pF, Capacitor_SMD:C_0402_1005Metric, F.Cu at (127.8, 70.2)
- added C23: 1.5pF, Capacitor_SMD:C_0402_1005Metric, F.Cu at (127.6, 73.8)
- added C24: C, Capacitor_SMD:C_0402_1005Metric, F.Cu at (161.2, 101.0)
- added C38: C, Capacitor_SMD:C_0402_1005Metric, F.Cu at (118.6, 76.6)
- added C39: C, Capacitor_SMD:C_0402_1005Metric, F.Cu at (118.6, 80.6)
- added C40: C, Capacitor_SMD:C_0402_1005Metric, F.Cu at (142.6, 68.6)
- added C41: C, Capacitor_SMD:C_0402_1005Metric, F.Cu at (142.6, 70.6)
- added C43: 10uF, Capacitor_SMD:C_0603_1608Metric, F.Cu at (206.2, 96.0)
- added C44: 10uF, Capacitor_SMD:C_0603_1608Metric, F.Cu at (206.2, 98.5)
- added C45: 10uF, Capacitor_SMD:C_0603_1608Metric, F.Cu at (206.2, 101.0)
- added D2: CHG_STATUS, LED_SMD:LED_0402_1005Metric, F.Cu at (142.1, 119.2)
- added J5: ESP_ANT, Connector_Coaxial:U.FL_Molex_MCRF_73412-0110_Vertical, F.Cu at (131.6, 71.2)
- added J6: GPS_ANT, Connector_Coaxial:U.FL_Molex_MCRF_73412-0110_Vertical, F.Cu at (169.9, 102.7)
- added JP1: BOOT, Jumper:SolderJumper-2_P1.3mm_Open_RoundedPad1.0x1.5mm, F.Cu at (178.8, 91.4)
- added L1: 2.7nH, Inductor_SMD:L_0402_1005Metric, F.Cu at (126.0, 72.0)
- added L3: 2nH, Inductor_SMD:L_0402_1005Metric, F.Cu at (140.4, 84.0)
- added Q1: BC818, Package_TO_SOT_SMD:SOT-23, F.Cu at (159.1, 50.0)
- added R10: 10k, Resistor_SMD:R_0402_1005Metric, F.Cu at (143.3, 88.0)
- added R17: 0, Resistor_SMD:R_0402_1005Metric, F.Cu at (146.2, 86.0)
- added R37: R, Resistor_SMD:R_0402_1005Metric, F.Cu at (118.6, 78.6)
- added R38: 10, Resistor_SMD:R_0603_1608Metric, F.Cu at (200.2, 107.6)
- added R39: 1k, Resistor_SMD:R_0402_1005Metric, F.Cu at (196.7, 109.3)
- added R40: 100, Resistor_SMD:R_0402_1005Metric, F.Cu at (196.7, 111.3)
- added U4: TPS63001, Package_SON:Texas_DRC0010J_ThermalVias, F.Cu at (188.2, 97.8)
- added Y1: 40MHz(10ppm), Crystal:Crystal_SMD_3225-4Pin_3.2x2.5mm, F.Cu at (131.4, 76.8)
- added Y2: 32.768kHz, Crystal:Crystal_SMD_3215-2Pin_3.2x1.5mm, F.Cu at (116.6, 78.6)
- C13, C14, D3, R11, R30, R32, R4, R5, R6, R7, R8, U1: moved to F.Cu
- C3: footprint Capacitor_SMD:C_0402_1005Metric -> Capacitor_SMD:C_0603_1608Metric
- TP3: value BATT- -> Conn_B-
- TP4: value BATT+ -> Conn_B+
- U2: value MAX-M10M -> MAX-M10S
- moved C14 72.6 mm to (176.6, 104.5), turned to 0 degrees
- moved U7 65.8 mm to (173.3, 68.0), turned to 0 degrees
- moved U1 64.4 mm to (156.8, 112.5), turned to 0 degrees
- moved D3 61.5 mm to (165.4, 104.9), turned to 0 degrees
- moved TP3 60.8 mm to (178.5, 76.1), turned to 0 degrees
- moved U10 59.2 mm to (172.4, 78.7), turned to 180 degrees
- moved C13 58.4 mm to (158.3, 97.0), turned to 0 degrees
- moved TP4 56.8 mm to (178.5, 80.6), turned to 0 degrees
- moved MK1 50.2 mm to (178.9, 87.1), turned to 0 degrees
- moved R32 48.2 mm to (152.0, 84.0), turned to 0 degrees
- moved C15 48.0 mm to (176.6, 106.2), turned to 0 degrees
- moved R8 42.2 mm to (143.3, 84.0), turned to 0 degrees
- moved C4 41.3 mm to (174.1, 102.8), turned to 0 degrees
- moved R7 39.8 mm to (143.3, 82.1), turned to 0 degrees
- moved R6 38.8 mm to (140.4, 96.0), turned to 0 degrees
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Connections:
- net /GPIO47 renamed /BTN1
- net /GPIO48 renamed /BTN2
- net /SPI2_CS0 renamed /DISP_CS
- net Net-(U8-GPIO46) renamed /DISP_RESET
- R31 pad 1: /GPIO_45 -> /GPS_INT
- R33 pad 1: /I2C1_SCL -> /I2C0_SCL
- R34 pad 1: /I2C1_SDA -> /I2C0_SDA
- U11 pad 13: /I2C1_SCL -> /I2C0_SCL
- U11 pad 14: /I2C1_SDA -> /I2C0_SDA
- U2 pad 11: unconnected-(U2-RF_IN-Pad11) -> Net-(U2-RF_IN)
- U2 pad 16: unconnected-(U2-SDA-Pad16) -> /I2C1_SDA
- U2 pad 17: unconnected-(U2-SCL-Pad17) -> /I2C1_SCL
- U2 pad 5: unconnected-(U2-EXTINT-Pad5) -> /GPS_INT
- U7 pad 17: +1V8 -> +5V
- U7 pad 4: +1V8 -> +5V
- U8 pad 1: Net-(U8-LNA_IN) -> /ESP_ANT
- U8 pad 10: unconnected-(U8-GPIO5-Pad10) -> /BAT_STAT2
- U8 pad 11: unconnected-(U8-GPIO6-Pad11) -> /MIC_WS
- U8 pad 12: unconnected-(U8-GPIO7-Pad12) -> /MIC_SCK
- U8 pad 13: unconnected-(U8-GPIO8-Pad13) -> /MIC_SD
- U8 pad 14: /SPI2_ -> /BL_CTRL
- U8 pad 16: /SPI2_ -> /DISP_MOSI
- U8 pad 17: /SPI2_ -> /DISP_CLK
- U8 pad 18: /SPI2_ -> /DISP_DC
- U8 pad 19: /SPI2_ -> /TP_INT
- U8 pad 21: unconnected-(U8-XTAL_32K_P-Pad21) -> /RTC_P
- U8 pad 22: unconnected-(U8-XTAL_32K_N-Pad22) -> /RTC_N
- U8 pad 23: unconnected-(U8-GPIO17-Pad23) -> /HBT_INT
- U8 pad 24: unconnected-(U8-GPIO18-Pad24) -> /IMU_INT2
- U8 pad 25: unconnected-(U8-GPIO19-Pad25) -> /USB_DM
- U8 pad 26: unconnected-(U8-GPIO20-Pad26) -> /USB_DM
- U8 pad 27: unconnected-(U8-GPIO21-Pad27) -> /IMU_Wakeup
- U8 pad 43: unconnected-(U8-GPIO38-Pad43) -> /LED_EN
- U8 pad 44: /GPIO39 -> /SD_D0
- U8 pad 45: /GPIO40 -> /SD_D1
- U8 pad 47: /GPIO41 -> /SD_D2
- U8 pad 48: /GPIO42 -> /SD_D3
- U8 pad 49: unconnected-(U8-U0TXD-Pad49) -> /SD_CLK
- U8 pad 5: /I2C1_SCL -> /I2C0_SCL
- U8 pad 50: unconnected-(U8-U0RXD-Pad50) -> /SD_CMD
- U8 pad 51: /GPIO_45 -> /GPS_INT
- U8 pad 53: unconnected-(U8-XTAL_N-Pad53) -> /CLK_N
- U8 pad 54: unconnected-(U8-XTAL_P-Pad54) -> /CLK_P
- U8 pad 6: /I2C1_SDA -> /I2C0_SDA
- U8 pad 7: unconnected-(U8-GPIO2-Pad7) -> /I2C1_SCL
- U8 pad 8: unconnected-(U8-GPIO3-Pad8) -> /I2C1_SDA
- U8 pad 9: unconnected-(U8-GPIO4-Pad9) -> /BAT_STAT1
Other:
- outline, holes or cut-outs redrawn
