File: cad/watch_pcb/watch_pcb.kicad_sch (KiCad schematic)
At the start: 96 parts, among them J1 DISPLAY, J2 Micro_SD_Card, J3 BATTERY, J4 USB_C_Receptacle, U1 LIS3MDL, U10 MX25LM51245GXDI00, U11 LSM6DSV16XTR, U2 MAX-M10M, U3 AMS1117-3.3, U4 FT231XQ, U5 AP131-18, U6 MAX30102, U7 MCP73871-2AA, U8 ESP32-S3, U9 S80KS5123GABHI020

Commit message: more
Parts:
- removed C16: 4.7uF, symbol Device:C_Small
- removed C17, C21: 100nF, symbol Device:C_Small
- removed J3: BATTERY, symbol Connector_Generic:Conn_01x02
- removed R10: 5.1k, symbol Device:R
- removed R17: 499, symbol Device:R
- removed U4: FT231XQ, Package_DFN_QFN:QFN-20-1EP_4x4mm_P0.5mm_EP2.5x2.5mm, symbol Interface_USB:FT231XQ
- added TP1: BOOT, TestPoint:TestPoint_Pad_D2.0mm, symbol Connector:TestPoint_Small
- added TP2: GND, TestPoint:TestPoint_Pad_2.0x2.0mm, symbol Connector:TestPoint_Small
- added TP3: BATT-, TestPoint:TestPoint_Pad_2.5x2.5mm, symbol Connector:TestPoint_Small
- added TP4: BATT+, TestPoint:TestPoint_Pad_D2.5mm, symbol Connector:TestPoint_Small
- C1, C19, C2, C20, C9: footprint (none) -> Capacitor_SMD:C_0603_1608Metric
- C10, C11, C14, C15, C26, C27, C30, C31, C32, C33, C36, C37, C4, C7, C8: footprint (none) -> Capacitor_SMD:C_0201_0603Metric
- C12, C13, C18, C25, C28, C29, C3, C34, C35, C5, C6: footprint (none) -> Capacitor_SMD:C_0402_1005Metric
- J2: footprint (none) -> 5033981892:MOLEX_503398-1892
- J4: footprint Inset USB-C:CU3024PAAHLR001-NH_CVI -> DX07B024JJ1R1500:JAE_DX07B024JJ1R1500
- R1, R11, R12, R13, R14, R15, R16, R18, R19, R2, R20, R21, R22, R23, R24, R25, R26, R27, R28, R29, R3, R30, R31, R32, R35, R36, R4, R5, R6, R7, R8: footprint (none) -> Resistor_SMD:R_0402_1005Metric
- R33, R34: value R -> 2k; footprint (none) -> Resistor_SMD:R_0402_1005Metric
- R9: value 5.1k -> 10k; footprint (none) -> Resistor_SMD:R_0402_1005Metric
- U10: footprint CSP24_6X8X1.2_MAC -> MX25UM51245G:CSP24_6X8X1.2_MAC
- U11: footprint LGA14L_LSM6_STM -> LSM6DSV16XTR:LGA14L_LSM6_STM
- U9: footprint PG-BGA-24-801 -> S80KS5123GABHI020:PG-BGA-24-801
Connections:
- net GND: now also R9.2, TP2.1, TP3.1
- net I2C1_SCL: now also TP1.1
- net USB_DM: no longer R9.1
- net BATT+: now reaches C20.1, U7.14 (V_{BAT}), U7.15 (V_{BAT}), U7.16 (V_{BAT_SENSE})
- net BATT+: now also TP4.1
- net at U8.52 (GPIO46): now also R9.1
- net UART_MOSI: no longer names the net of U8.50 (U0RXD)
- no-connect marks 26 -> 16
Other:
- note added: "LED audio driver buttons"
- note removed: "LED speaker? buttons"
- moved on the sheet: AE1, J1, R31, U2

Commit message: idk some stuff
Parts:
- removed AE1: Antenna_Dipole, RF_Antenna:Texas_SWRA117D_2.4GHz_Right, symbol Device:Antenna_Dipole
- removed C2: 22uF, Capacitor_SMD:C_0603_1608Metric, symbol Device:C_Small
- removed TP1: BOOT, TestPoint:TestPoint_Pad_D2.0mm, symbol Connector:TestPoint_Small
- removed TP2: GND, TestPoint:TestPoint_Pad_2.0x2.0mm, symbol Connector:TestPoint_Small
- removed U2: MAX-M10M, RF_GPS:ublox_MAX, symbol RF_GPS:MAX-M10M
- removed U3: AMS1117-3.3, Package_TO_SOT_SMD:SOT-223-3_TabPin2, symbol Regulator_Linear:AMS1117-3.3
- added C16: 100nF, Capacitor_SMD:C_0201_0603Metric, symbol Device:C_Small
- added C17: 1uF, Capacitor_SMD:C_0402_1005Metric, symbol Device:C_Small
- added C21, C38, C39, C40, C41: C, Capacitor_SMD:C_0402_1005Metric, symbol Device:C_Small
- added C42: 100nF, symbol Device:C_Small
- added C43, C44, C45: 10uF, Capacitor_SMD:C_0603_1608Metric, symbol Device:C_Small
- added J3: Conn_01x06_Socket, symbol Connector:Conn_01x06_Socket
- added J5: ESP_ANT, Connector_Coaxial:U.FL_Molex_MCRF_73412-0110_Vertical, symbol Connector:Conn_Coaxial_Small
- added J6: GPS_ANT, Connector_Coaxial:U.FL_Molex_MCRF_73412-0110_Vertical, symbol Connector:Conn_Coaxial_Small
- added JP1: BOOT, Jumper:SolderJumper-2_P1.3mm_Open_RoundedPad1.0x1.5mm, symbol Jumper:SolderJumper_2_Open
- added LS1: Speaker, symbol Device:Speaker
- added Q1: BC818, Package_TO_SOT_SMD:SOT-23, symbol Transistor_BJT:BC818
- added R10: 10k, Resistor_SMD:R_0402_1005Metric, symbol Device:R
- added R17: 0, Resistor_SMD:R_0402_1005Metric, symbol Device:R
- added R37: R, Resistor_SMD:R_0402_1005Metric, symbol Device:R
- added R38: 10, Resistor_SMD:R_0603_1608Metric, symbol Device:R
- added R39: 1k, Resistor_SMD:R_0402_1005Metric, symbol Device:R
- added R40: 100, Resistor_SMD:R_0402_1005Metric, symbol Device:R
- added U12: LC709203FQH-01TWG, Package_DFN_QFN:WDFN-8-1EP_4x3mm_P0.65mm_EP2.4x1.8mm, symbol Battery_Management:LC709203FQH-01TWG
- added U2: MAX-M10S, RF_GPS:ublox_MAX, symbol RF_GPS:MAX-M10S
- added U3: MAX17261xxWL, Package_BGA:Maxim_WLP-9_1.595x1.415_Layout3x3_P0.4mm_Ball0.27mm_Pad0.25mm_NSMD, symbol Battery_Management:MAX17261xxWL
- added U4: TPS63001, Package_SON:Texas_DRC0010J_ThermalVias, symbol Regulator_Switching:TPS63001
- added Y1: 40MHz(10ppm), Crystal:Crystal_SMD_3225-4Pin_3.2x2.5mm, symbol Device:Crystal_GND24_Small
- added Y2: 32.768kHz, Crystal:Crystal_SMD_3215-2Pin_3.2x1.5mm, symbol Device:Crystal_Small
- C1: value 22uF -> 1uF; footprint Capacitor_SMD:C_0603_1608Metric -> (none)
- C22, C23: value C -> 1.5pF; footprint (none) -> Capacitor_SMD:C_0402_1005Metric
- C24: footprint (none) -> Capacitor_SMD:C_0402_1005Metric
- C3: footprint Capacitor_SMD:C_0402_1005Metric -> Capacitor_SMD:C_0603_1608Metric
- D2: footprint (none) -> LED_SMD:LED_0402_1005Metric
- J1: footprint Connector_FFC-FPC:Hirose_FH12-18S-0.5SH_1x18-1MP_P0.50mm_Horizontal -> Connector_FFC-FPC:TE_1-1734839-8_1x18-1MP_P0.5mm_Horizontal
- L1: value L -> 2.7nH; footprint (none) -> Inductor_SMD:L_0402_1005Metric
- L2: value L -> 2.2uH
- L3: footprint (none) -> Inductor_SMD:L_0402_1005Metric
- TP3: value BATT- -> Conn_B-
- TP4: value BATT+ -> Conn_B+
Connections:
- net GPIO39 is gone; now on net SD_D0: U8.44 (MTCK)
- net GPIO40 is gone; now on net SD_D1: U8.45 (MTDO)
- net GPIO41 is gone; now on net SD_D2: U8.47 (MTDI)
- net GPIO42 is gone; now on net SD_D3: U8.48 (MTMS)
- net SPI2_CS0 is gone; now on net DISP_CS: U8.15 (GPIO10)
- net +1V8: no longer U7.17 (CE), U7.4 (PROG2)
- net +3V3: now also J1.17 (Pin_17), J1.3 (Pin_3), J1.4 (Pin_4), C16.2, C17.2, C44.2, C45.2, J3.1 (Pin_1), U2.7 (VCC_IO), U2.8 (VCC), U4.1 (VOUT), U4.10 (FB)
- net +5V: now also U7.17 (CE), U7.4 (PROG2), R10.1
- net +BATT: now also C43.2, R40.1, U4.5 (VIN); no longer C1.1
- net BATT+: now also C1.1, U12.3 (V_{DD})
- net CPU_EN: now also J3.2 (Pin_2)
- net GND: now also J1.1 (Pin_1), J1.12 (Pin_12), J1.18 (Pin_18), J1.5 (Pin_5), J1.6 (Pin_6), C16.1, C17.1, C21.2, C38.1, C39.1, C40.1, C41.2, C42.2, C43.1, C44.1, C45.1, J3.6 (Pin_6), J5.2 (Ext), J6.2 (Ext), JP1.1 (A), Q1.2 (E), R10.2, U12.1 (TEST), U12.2 (V_{SS}), U12.9 (EP), U2.1 (GND), U2.10 (GND), U2.12 (GND), U4.11 (PGND), U4.3 (PGND), U4.9 (GND), Y1.2, Y1.4
- net HBT_INT: now also U8.23 (GPIO17)
- net I2C1_SCL: now also J1.13 (Pin_13), U8.7 (GPIO2), U12.8 (SCL), U2.17 (SCL); no longer R33.1, U11.13 (SCL), U8.5 (GPIO0)
- net I2C1_SDA: now also J1.14 (Pin_14), U8.8 (GPIO3), U12.7 (SDA), U2.16 (SDA); no longer R34.1, U11.14 (SDA), U8.6 (GPIO1)
- net IMU_INT2: now also U8.24 (GPIO18)
- net IMU_Wakeup: now also U8.27 (GPIO21)
- net MIC_SCK: now also U8.12 (GPIO7)
- net MIC_SD: now also U8.13 (GPIO8)
- net MIC_WS: now also U8.11 (GPIO6)
- net SD_CLK: now also U8.49 (U0TXD)
- net SD_CMD: now also U8.50 (U0RXD)
- net USB_DM: now also U8.25 (GPIO19), U8.26 (GPIO20)
- net at L2.1: now also U4.4 (L1); no longer C24.1
- net DISP_MOSI: now reaches J1.10 (Pin_10)
- net DISP_MOSI: now also U8.16 (GPIO11)
- net DISP_RESET: now reaches J1.11 (Pin_11)
- net DISP_RESET: now also J1.15 (Pin_15), R9.1, U8.52 (GPIO46)
- net TP_INT: now reaches J1.16 (Pin_16)
- net TP_INT: now also U8.19 (GPIO14)
- net LEDK: now reaches J1.2 (Pin_2)
- net LEDK: now also R38.2
- net DISP_DC: now reaches J1.7 (Pin_7)
- net DISP_DC: now also U8.18 (GPIO13)
- net DISP_CS: now reaches J1.8 (Pin_8)
- net DISP_CLK: now reaches J1.9 (Pin_9)
- net DISP_CLK: now also U8.17 (GPIO12)
- net ESP_ANT: now reaches L1.2, U8.1 (LNA_IN)
- net ESP_ANT: now also C23.1; no longer C22.1
- net RTC_P: now reaches U8.21 (XTAL_32K_P)
- net RTC_P: now also C38.2, R37.1, Y2.2
- net RTC_N: now reaches U8.22 (XTAL_32K_N)
- net RTC_N: now also C39.2, R37.2, Y2.1
- net LED_EN: now reaches U8.43 (GPIO38)
- net LED_EN: now also J3.3 (Pin_3)
- net CLK_N: now reaches U8.53 (XTAL_N)
- net CLK_N: now also C40.2, Y1.3
- net CLK_P: now reaches U8.54 (XTAL_P)
- net CLK_P: now also C41.1, Y1.1
- removed net ANT: C23.1, L1.1, L2.2
- net GPIO47 renamed BTN1
- net BTN1: now also J3.4 (Pin_4)
- net GPIO48 renamed BTN2
- net BTN2: now also J3.5 (Pin_5)
- net GPIO_45 renamed GPS_INT
- net GPS_INT: now also U2.5 (EXTINT)
- removed net SPI2_: U8.14 (GPIO9), U8.16 (GPIO11), U8.17 (GPIO12), U8.18 (GPIO13), U8.19 (GPIO14)
- new net: C21.1, J6.1 (In), R17.2
- new net: C22.1, J5.1 (In), L1.1
- new net: L2.2, U4.2 (L2)
- new net: C42.1, R40.2, U4.6 (EN), U4.7 (PS/SYNC), U4.8 (VINA)
- new net: Q1.1 (B), R39.2
- new net: Q1.3 (C), R38.1
- new net: C24.1, R17.1, U2.11 (RF_IN)
- new net BL_CTRL: R39.1, U8.14 (GPIO9)
- new net I2C0_SCL: JP1.2 (B), R33.1, U11.13 (SCL), U8.5 (GPIO0)
- new net I2C0_SDA: R34.1, U11.14 (SDA), U8.6 (GPIO1)
- no-connect marks 16 -> 26
Other:
- note added: "1.7A"
- note added: "CM315D32768HZFT"
- note added: "FL4000157Z"
- note added: "GRM0335C1H1R5BA01D"
- note added: "LQP03TN2N7B02D"
- note added: "TODO: gps antenna black magic may not need pi?"
- note added: "VLF4012-2R2"
- note added: "battery measurement?"
- note added: "impedance match or something"
- note removed: "1A"
- note removed: "LED audio driver buttons"
- note removed: "Screen (fast)"
- note removed: "charging always enabled"
- moved on the sheet: J1, R9
