File: watch-pcb.kicad_sch (KiCad schematic)
At the start: 104 parts, among them J2 Micro_SD_Card, J3 Conn_01x06_Socket, J4 USB_C_Receptacle, J5 ESP_ANT, U1 LIS3MDL, U10 MX25LM51245GXDI00, U2 BQ25629RYKR, U3 DRV2605LYZFR, U4 BQ27427YZFR, U5 APS12808L-3OBMx, U6 MAX30102, U7 LSM6DSV16XTR, U8 ESP32-S3, Y1 40MHz(10ppm), Y2 32.768kHz

Commit message: display started
Parts:
- removed U3: DRV2605LYZFR, DRV2605L:YZF0009ADAD, symbol DRV2605LYZFR:DRV2605LYZFR
- removed U4: BQ27427YZFR, BQ27427YZFR:IC_BQ27427YZFR, symbol BQ27427YZFR:BQ27427YZFR
- added C12, C49: 100nF, Capacitor_SMD:C_0201_0603Metric, symbol Device:C_Small
- added C2, C36: 1uF, Capacitor_SMD:C_0201_0603Metric, symbol Device:C_Small
- added J1: TT143AMC12C, symbol custom-lib:TT143AMC12C
- added R14: 10k, symbol Device:R
- added U3: BQ27427YZFR, Package_BGA:Texas_DSBGA-9_1.4715x1.4715mm_Layout3x3_P0.5mm, symbol custom-lib:BQ27427YZFR
- added U9: DRV2605LYZFR, Package_BGA:Texas_DSBGA-9_1.4715x1.4715mm_Layout3x3_P0.5mm, symbol custom-lib:DRV2605LYZFR
- C16: value 100nF -> 1uF
- C18: value 1uF -> 100nF
- C43: value 2.2uF -> 1uF
- C5: value 1uF -> 2.2uF
Connections:
- net +3V3: now also C17.1, C18.2, C42.1, C43.1, C12.1, C36.2, C49.2, J1.1 (VDD), J1.19 (IOVCC), J1.20 (VDD), U3.C2 (SRX), U9.A1 (EN), U9.C2 (VDD); no longer C16.1, C18.1, C5.2
- net BAT+: now also C16.2, U3.C3 (BAT); no longer C42.1
- net BAT_LOW: now also U3.A1 (GPOUT)
- net GND: now also C16.1, C18.1, C43.2, C12.2, C2.2, C36.1, C49.1, J1.10 (GND), J1.12 (GND), J1.18 (GND), J1.6 (GND), R14.1, U3.B2 (VSS), U3.C1 (VSS), U9.B1 (IN/TRIG), U9.B3 (GND); no longer C16.2, C18.2, C43.1
- net I2C1_SCL: now also J1.4 (SCL), U3.A3 (SCL), U9.C1 (SCL)
- net I2C1_SDA: now also J1.3 (SDA), U3.A2 (SDA), U9.B2 (SDA)
- net MTR_M: now also U9.C3 (OUT-)
- net MTR_P: now also U9.A3 (OUT+)
- new net: R14.2, U3.B1 (BIN)
- new net: C2.1, U9.A2 (REG)
- new net: C5.2, U3.B3 (VDD)
- new net TP_INT: J1.2 (INT)
- new net TP_RST: J1.5 (RST)

Commit message: finished schematic, verifying design and doing daughter board
Parts:
- removed C1: 1uF, Capacitor_SMD:C_0201_0603Metric, symbol Device:C_Small
- removed C21, C24, C37: 10uF, Capacitor_SMD:C_0201_0603Metric, symbol Device:C_Small
- removed C44: 1uF, symbol Device:C_Small
- removed C45: 100nF, symbol Device:C_Small
- removed D1: STAT, symbol Device:LED
- removed JP1: BOOT, Jumper:SolderJumper-2_P1.3mm_Open_RoundedPad1.0x1.5mm, symbol Jumper:SolderJumper_2_Open
- removed L2: 1uH, symbol Device:L
- removed R10, R13, R17, R3, R31, R33, R34, R35, R36, R41, R9: 10k, Resistor_SMD:R_0402_1005Metric, symbol Device:R
- removed R12: R, symbol Device:R
- removed TH1: Thermistor, symbol Device:Thermistor
- removed TP3: Conn_B-, TestPoint:TestPoint_Pad_2.5x2.5mm, symbol Connector:TestPoint_Small
- removed TP4: Conn_B+, TestPoint:TestPoint_Pad_D2.5mm, symbol Connector:TestPoint_Small
- removed U10: MX25LM51245GXDI00, MX25UM51245G:CSP24_6X8X1.2_MAC, symbol Custom_Flash:MX25LM51245GXDI00
- removed U2: BQ25629RYKR, BQ25628RYKR:IC_BQ25628RYKR, symbol BQ25628RYKR:BQ25628RYKR
- removed U5: APS12808L-3OBMx, custom-lib:BGA-24_6.0x8.0mm_Layout5x5_P1.0mm, symbol custom-lib:APS12808L-3OBMx
- added BT1: Battery, custom-lib:Battery_Connector, symbol Device:Battery
- added C12, C22: 22uF, symbol Device:C_Small
- added C14, C55, C58, C64, C74, C75, C78, C79, C9: 100nF, symbol Device:C_Small
- added C15, C56, C59, C63, C65, C72, C76: 1uF, symbol Device:C_Small
- added C16, C26, C27, C28, C29, C5, C7, C77, C80: 10uF, symbol Device:C_Small
- added C17, C18: 4.7uF, symbol Device:C_Small
- added C23: 47nF, symbol Device:C_Small
- added C66, C67, C68, C69: C, symbol Device:C_Small
- added C70, C71: 1.5pF, Capacitor_SMD:C_0201_0603Metric, symbol Device:C_Small
- added C73: 10nF, symbol Device:C_Small
- added D2: CHARGING, symbol Device:LED
- added D3: POWER GOOD, symbol Device:LED
- added J6: ESP_ANT, Connector_Coaxial:U.FL_Molex_MCRF_73412-0110_Vertical, symbol Connector:Conn_Coaxial_Small
- added JP2, JP3, JP4, JP5, JP8: GP6, Jumper:SolderJumper-3_P1.3mm_Open_RoundedPad1.0x1.5mm, symbol Jumper:SolderJumper_3_Open
- added JP6: RESET=LOW, Jumper:SolderJumper-2_P1.3mm_Open_RoundedPad1.0x1.5mm, symbol Jumper:SolderJumper_2_Open
- added L1: 1.5uH, symbol Device:L
- added L3, L4: 10uH, symbol Device:L
- added L5: 1uH, symbol Device:L
- added L7: 2.7nH, Inductor_SMD:L_0201_0603Metric, symbol Device:L
- added L8: 2nH, symbol Device:L
- added R21: R, PCM_Resistor_SMD_AKL:R_0402_1005Metric, symbol Device:R
- added R22: 5.1k, symbol Device:R
- added R39: 5.24k, symbol Device:R
- added R4: 180k, symbol Device:R
- added R40: 30.31, symbol Device:R
- added R42, R43, R44, R45, R46, R47, R48, R49, R50, R51, R52, R53, R54: 10k, symbol Device:R
- added R5, R6: 1M, symbol Device:R
- added R7: 1.5k, symbol Device:R
- added SW1: USB, symbol Switch:SW_Push_Dual
- added TH1: 103AT-2 10k, symbol Device:Thermistor_NTC
- added TP1: MTP_PWR, symbol Connector:TestPoint_Small
- added TP2: FLASH RESET, symbol Connector:TestPoint
- added TP3: RAM RESET, symbol Connector:TestPoint
- added TP4: ECS, symbol Connector:TestPoint
- added U10: APS12808L-3OBMx, custom-lib:BGA-24_6.0x8.0mm_Layout5x5_P1.0mm, symbol custom-lib:APS12808L-3OBMx
- added U12: ESP32-S3, Package_DFN_QFN:QFN-56-1EP_7x7mm_P0.4mm_EP4x4mm_ThermalVias, symbol MCU_Espressif:ESP32-S3
- added U2: TPS63021, custom-lib:Texas_VSON-14_3x4mm_ThermalPad, symbol custom-lib:TPS63021
- added U3: BQ25638, custom-lib:Texas_DSBGA-30_2.0x2.4mm_Layout5x6_P0.4mm, symbol custom-lib:BQ25638
- added U4: TPS65631W, Package_SON:WSON-10-1EP_2.5x2.5mm_P0.5mm_EP1.2x2mm_ThermalVias, symbol custom-lib:TPS65631W
- added U9: MX25LM51245GXDI00, custom-lib:BGA-24_6.0x8.0mm_Layout5x5_P1.0mm, symbol custom-lib:MX25LM51245GXDI00
- added Y3: 40MHz(10ppm), Crystal:Crystal_SMD_3225-4Pin_3.2x2.5mm, symbol Device:Crystal_GND24_Small
- added Y4: 32.768kHz, Crystal:Crystal_SMD_3215-2Pin_3.2x1.5mm, symbol Device:Crystal_Small
- C1: renamed from C41; footprint Capacitor_SMD:C_0402_1005Metric -> (none)
- C10: renamed from C38; footprint Capacitor_SMD:C_0402_1005Metric -> (none)
- C11: renamed from C39; footprint Capacitor_SMD:C_0402_1005Metric -> (none)
- C13: renamed from C22; footprint Capacitor_SMD:C_0402_1005Metric -> (none)
- C19: value 47nF -> 22uF; footprint Capacitor_SMD:C_0201_0603Metric -> (none)
- C2: renamed from C40; footprint Capacitor_SMD:C_0402_1005Metric -> (none)
- C20: value 4.7uF -> 10uF; footprint Capacitor_SMD:C_0201_0603Metric -> (none)
- C21: renamed from C23; footprint Capacitor_SMD:C_0402_1005Metric -> (none)
- C24: renamed from C42; footprint Capacitor_SMD:C_0201_0603Metric -> (none)
- C25: renamed from C18; footprint Capacitor_SMD:C_0201_0603Metric -> (none)
- C3: renamed from C12; footprint Capacitor_SMD:C_0201_0603Metric -> (none)
- C30: renamed from C43; footprint Capacitor_SMD:C_0201_0603Metric -> (none)
- C31: renamed from C49; footprint Capacitor_SMD:C_0201_0603Metric -> (none)
- C32: renamed from C29; footprint Capacitor_SMD:C_0402_1005Metric -> (none)
- C33: renamed from C16; footprint Capacitor_SMD:C_0201_0603Metric -> (none)
- C34: renamed from C30; footprint Capacitor_SMD:C_0201_0603Metric -> (none)
- C35: renamed from C25; footprint Capacitor_SMD:C_0402_1005Metric -> (none)
- C36: renamed from C28; footprint Capacitor_SMD:C_0402_1005Metric -> (none)
- C37: renamed from C5; footprint Capacitor_SMD:C_0201_0603Metric -> (none)
- C38: renamed from C26; footprint Capacitor_SMD:C_0201_0603Metric -> (none)
- C39: renamed from C27; footprint Capacitor_SMD:C_0201_0603Metric -> (none)
- C4: renamed from C36; footprint Capacitor_SMD:C_0201_0603Metric -> (none)
- C40: renamed from C31; footprint Capacitor_SMD:C_0201_0603Metric -> (none)
- C41: renamed from C32; footprint Capacitor_SMD:C_0201_0603Metric -> (none)
- C42: renamed from C33; footprint Capacitor_SMD:C_0201_0603Metric -> (none)
- C43: renamed from C6; footprint Capacitor_SMD:C_0402_1005Metric -> (none)
- C44: renamed from C7; footprint Capacitor_SMD:C_0201_0603Metric -> (none)
- C45: renamed from C34; footprint Capacitor_SMD:C_0402_1005Metric -> (none)
- C46: renamed from C35; footprint Capacitor_SMD:C_0402_1005Metric -> (none)
- C47: renamed from C15; footprint Capacitor_SMD:C_0201_0603Metric -> (none)
- C48: renamed from C17; footprint Capacitor_SMD:C_0201_0603Metric -> (none)
- C49: renamed from C9; footprint Capacitor_SMD:C_0603_1608Metric -> (none)
- C50: renamed from C8; footprint Capacitor_SMD:C_0201_0603Metric -> (none)
- C51: renamed from C4; footprint Capacitor_SMD:C_0201_0603Metric -> (none)
- C54: renamed from C10; footprint Capacitor_SMD:C_0201_0603Metric -> (none)
- C57: renamed from C13; footprint Capacitor_SMD:C_0402_1005Metric -> (none)
- C6: renamed from C2; footprint Capacitor_SMD:C_0201_0603Metric -> (none)
- C60: renamed from C46; footprint Capacitor_SMD:C_0201_0603Metric -> (none)
- C61: renamed from C47; footprint Capacitor_SMD:C_0201_0603Metric -> (none)
- C62: renamed from C48; footprint Capacitor_SMD:C_0201_0603Metric -> (none)
- C8: renamed from C14; footprint Capacitor_SMD:C_0201_0603Metric -> (none)
- J1: renamed from J4; footprint DX07B024JJ1R1500:JAE_DX07B024JJ1R1500 -> Connector_USB:USB_C_Receptacle_GCT_USB4105-xx-A_16P_TopMnt_Horizontal
- L2: renamed from L1; footprint Inductor_SMD:L_0402_1005Metric -> (none)
- L6: renamed from L3; footprint Inductor_SMD:L_0402_1005Metric -> (none)
- R1, R2, R20: footprint Resistor_SMD:R_0402_1005Metric -> (none)
- R10: renamed from R26; footprint Resistor_SMD:R_0402_1005Metric -> (none)
- R11: renamed from R23; footprint Resistor_SMD:R_0402_1005Metric -> (none)
- R12: renamed from R22; footprint Resistor_SMD:R_0402_1005Metric -> (none)
- R13: renamed from R21; footprint Resistor_SMD:R_0402_1005Metric -> (none)
- R14: renamed from R30; footprint Resistor_SMD:R_0402_1005Metric -> (none)
- R15: renamed from R29; footprint Resistor_SMD:R_0402_1005Metric -> (none)
- R16: renamed from R28; footprint Resistor_SMD:R_0402_1005Metric -> (none)
- R17: renamed from R25; footprint Resistor_SMD:R_0402_1005Metric -> (none)
- R18: renamed from R24; footprint Resistor_SMD:R_0402_1005Metric -> (none)
- R3: renamed from R37; footprint Resistor_SMD:R_0402_1005Metric -> (none)
- R32: renamed from R11; footprint Resistor_SMD:R_0402_1005Metric -> (none)
- R33: renamed from R32; footprint Resistor_SMD:R_0402_1005Metric -> (none)
- R34: renamed from R8; footprint Resistor_SMD:R_0402_1005Metric -> (none)
- R35: renamed from R7; footprint Resistor_SMD:R_0402_1005Metric -> (none)
- R36: renamed from R5; footprint Resistor_SMD:R_0402_1005Metric -> (none)
- R37: renamed from R4; footprint Resistor_SMD:R_0402_1005Metric -> (none)
- R38: renamed from R6; footprint Resistor_SMD:R_0402_1005Metric -> (none)
- R8: renamed from R18; footprint Resistor_SMD:R_0402_1005Metric -> (none)
- R9: renamed from R27; footprint Resistor_SMD:R_0402_1005Metric -> (none)
- U5: renamed from U8; footprint ESP32-S3:IC_ESP32-S3 -> Package_DFN_QFN:QFN-56-1EP_7x7mm_P0.4mm_EP4x4mm_ThermalVias
- renumbered C11 to C52, C3 to C53, D3 to D1, J5 to J2, J1 to J3, J3 to J4, J2 to J5, R14 to R19, U9 to U1, U7 to U11, U3 to U6, U6 to U7, U1 to U8
Connections:
- net REGN is gone; now on net GND: C20.1
- net +1V8: now also C36.2, C39.2, U5.29 (VDD_SPI)
- net +3V3: now also C19.2, C20.2, C12.2, C14.1, C22.2, C55.1, C56.1, C58.1, C59.1, C72.2, C73.2, C75.1, C76.1, C77.1, C80.1, L4.1, L8.2, R22.2, R42.1, R43.1, R44.2, R45.2, R46.2, R47.2, R48.2, R49.2, R5.2, R50.2, R51.2, R52.2, R53.2, R54.2, R6.1, U10.B4 (VDD), U10.D1 (VDDQ), U10.E4 (VDDQ), U12.55 (VDDA1), U12.56 (VDDA2), U2.4 (VOUT), U2.5 (VOUT), U4.10 (PVIN), U4.9 (AVIN), U9.B4 (VCC), U9.D1 (VCCQ), U9.E4 (VCCQ)
- net +5V: now also C15.2, U3.A1 (VBUS), U3.B1 (VBUS)
- net BAT+: now also BT1.1 (+), C18.2, U3.E1 (BAT), U3.E2 (BAT), U3.E3 (BAT), U3.F1 (BATP)
- net BAT_LOW: now also U5.10 (GPIO5), R52.1; no longer U5.43 (GPIO38)
- net BTN1: now also U12.51 (GPIO45)
- net CHG_INT: now also U5.9 (GPIO4), R51.1, U3.F5 (INT); no longer U5.51 (GPIO45)
- net CLK_N: now also C67.2, U12.53 (XTAL_N), Y3.3
- net CLK_P: now also C66.1, U12.54 (XTAL_P), Y3.1
- net CPU_EN: no longer J4.2 (Pin_2)
- net ESP_ANT: now also C71.1, L7.2, U12.1 (LNA_IN)
- net GND: now also C19.1, BT1.2 (-), C12.1, C14.2, C15.1, C16.1, C17.1, C18.1, C22.1, C26.1, C27.2, C28.1, C29.2, C5.2, C55.2, C56.2, C58.2, C59.2, C63.1, C64.1, C65.2, C66.2, C67.1, C68.1, C69.1, C7.1, C70.2, C71.2, C72.1, C73.1, C78.1, C79.1, C9.1, J6.2 (Ext), JP6.1 (A), L3.1, R4.1, R40.1, R7.1, SW1.2, SW1.4, TH1.1, U10.B3 (VSS), U10.C1 (VSSQ), U10.E5 (VSSQ), U12.57 (GND), U2.15 (PGND), U2.2 (GND), U3.A4 (PGND), U3.B4 (PGND), U3.C4 (PGND), U3.C5 (ADCIN), U3.F2 (CE), U4.11 (GND), U4.2 (PGND), U4.5 (AGND), U9.B3 (GND), U9.C1 (VSSQ), U9.E5 (VSSQ), Y3.2, Y3.4; no longer C20.2
- net HBT_INT: now also JP4.3 (B), JP8.3 (B), R53.1; no longer U5.23 (GPIO17)
- net I2C0_SCL: now also R45.1, SW1.1, U12.5 (GPIO0)
- net I2C0_SDA: now also R44.1, U12.6 (GPIO1)
- net I2C1_SCL: now also R47.1, U12.7 (GPIO2), U3.D5 (SCL)
- net I2C1_SDA: now also R46.1, U12.8 (GPIO3), U3.E5 (SDA)
- net IMU_SCL: now also R49.1
- net IMU_SDA: now also R48.1
- net IMU_Wakeup: now also U5.23 (GPIO17); no longer U5.27 (GPIO21)
- net MAG_INT: now also JP3.1 (A); no longer U5.24 (GPIO18)
- net MEM_CLK: now also U10.B2 (CLK), U9.B2 (SCLK)
- net MEM_CS0: now also U9.C2 (CS#)
- net MEM_CS1: now also U10.A3 (CE#)
- net MEM_D0: now also U10.D3 (ADQ0), U9.D3 (SIO0)
- net MEM_D1: now also U10.D2 (ADQ1), U9.D2 (SIO1)
- net MEM_D2: now also U10.C4 (ADQ2), U9.C4 (SIO2)
- net MEM_D3: now also U10.D4 (ADQ3), U9.D4 (SIO3)
- net MEM_D4: now also U10.D5 (ADQ4), U9.D5 (SIO4)
- net MEM_D5: now also U10.E3 (ADQ5), U9.E3 (SIO5)
- net MEM_D6: now also U10.E2 (ADQ6), U9.E2 (SIO6)
- net MEM_D7: now also U10.E1 (ADQ7), U9.E1 (SIO7)
- net MEM_DQS: now also U10.C3 (DQS/DM), U9.C3 (DQS)
- net MIC_SCK: now also U5.43 (GPIO38); no longer U5.10 (GPIO5)
- net MIC_SD: now also U5.52 (GPIO46); no longer U5.11 (GPIO6)
- net MIC_WS: now also U5.12 (GPIO7); no longer U5.9 (GPIO4)
- net POWER_BTN: now also J4.2 (Pin_2), U3.D4 (QON)
- net RTC_N: now also C69.2, R21.2, U12.22 (XTAL_32K_N), Y4.1
- net RTC_P: now also C68.2, R21.1, U12.21 (XTAL_32K_P), Y4.2
- net TP_INT: now also JP5.1 (A)
- net TP_RST: now also JP2.1 (A)
- net USB_DM: now also U12.25 (GPIO19); no longer U5.26 (GPIO20)
- net USB_DP: now also U5.26 (GPIO20), U12.26 (GPIO20)
- net VBUS: now also C27.1, C29.1, C5.1, C7.2, C9.2, D2.2 (A), D3.2 (A), L5.2, U2.1 (VINA), U2.10 (VIN), U2.11 (VIN), U2.12 (EN), U2.13 (PS/SYNC), U3.D1 (SYS), U3.D2 (SYS), U3.D3 (SYS)
- net at R20.2: now also C65.1, U12.4 (CHIP_PU)
- net FSPICLK: now reaches J3.11 (SCL)
- net FSPICLK: now also U5.17 (GPIO12)
- net FSPIQ: now reaches J3.13 (D1)
- net FSPIQ: now also U5.18 (GPIO13)
- net FSPIWP: now reaches J3.14 (D2)
- net FSPIWP: now also U5.19 (GPIO14)
- net DISP_RST: now reaches J3.15 (RST)
- net DISP_RST: now also JP4.1 (A), JP8.1 (A), R54.1
- net DISP_TE: now reaches J3.16 (TE)
- net DISP_TE: now also U5.13 (GPIO8)
- net SWIRE: now reaches J3.17 (SWIRE)
- net SWIRE: now also U4.6 (CTRL)
- net AMOLED_P: now reaches J3.22 (ELVDD)
- net AMOLED_P: now also C28.2, U4.3 (OUTP), U4.4 (FBS)
- net AMOLED_N: now reaches J3.23 (ELVSS)
- net AMOLED_N: now also C26.2, U4.7 (OUTN)
- net at J3.24 (MTP_PWR): now also TP1.1
- net FSPICS0: now reaches J3.7 (CS)
- net FSPICS0: now also U5.15 (GPIO10)
- net FSPID: now reaches J3.8 (D0)
- net FSPID: now also U5.16 (GPIO11)
- net FSPIHD: now reaches J3.9 (D3)
- net FSPIHD: now also U5.14 (GPIO9)
- net IMU_INT2: no longer names the net of U11.9 (INT2)
- net IMU_INT2: no longer U5.52 (GPIO46)
- net LED_EN: no longer names the net of J4.3 (Pin_3)
- removed net VMEM: C36.2, C39.2, R20.1, U5.29 (VDD_SPI)
- new net: C23.1, U3.B5 (BTST)
- new net: C23.2, L5.1, U3.A3 (SW), U3.B3 (SW), U3.C3 (SW)
- new net: R42.2, TP2.1, U9.A4 (RESET#)
- new net: R43.2, TP3.1, U10.A4 (RST#)
- new net: C16.2, U3.A2 (PMID), U3.B2 (PMID)
- new net: R7.2, U3.F3 (ILIM)
- new net: C74.2, C75.2, C76.2, C77.2, C80.2
- new net: C74.1, L8.1, U12.2 (VDD3P3), U12.3 (VDD3P3__1)
- new net: C78.2, C79.2, U12.20 (VDD3P3_RTC), U12.46 (VDD3P3_CPU)
- new net: C63.2, C64.2, U12.29 (VDD_SPI)
- new net: D3.1 (K), U3.C2 (PG)
- new net: L3.2, U4.8 (SWN)
- new net: R4.2, R5.1, U2.3 (FB)
- new net: C17.2, U3.A5 (REGN)
- new net: L1.1, U2.8 (L1), U2.9 (L1)
- new net: L1.2, U2.6 (L2), U2.7 (L2)
- new net: C70.1, J6.1 (In), L7.1
- new net: D2.1 (K), U3.C1 (STAT)
- new net: R39.1, R40.2, TH1.2, U3.E4 (TS)
- new net: R39.2, U3.F4 (TS_BIAS)
- new net: L4.2, U4.1 (SWP)
- new net: TP4.1, U9.A5 (ECS#)
- new net CPU_RST: JP6.2 (B), R20.1, R22.1
- new net FLASH_ECS: JP2.3 (B)
- new net FLASH_RST: JP5.3 (B), R50.1
- new net GP18: JP5.2 (C), U5.24 (GPIO18)
- new net GP21: JP3.2 (C), U5.27 (GPIO21)
- new net GP45: JP4.2 (C), JP8.2 (C), U5.51 (GPIO45)
- new net GP46: SW1.3, U12.52 (GPIO46)
- new net GP6: JP2.2 (C), U5.11 (GPIO6)
- new net PWR_GOOD: R6.2, U2.14 (PG)
- new net RAM_RST: JP3.3 (B)
Other:
- note added: "16MB PSRAM, 120MHz(133) DDR OPI"
- note added: "64MB NOR Flash, 120MHz(133) DDR OPI"
- note added: "GOOD"
- note added: "gp44 gp43"
- note added: "recalculate R for 0 1 imu"
- note added: "std"
- note removed: "103AT NTC"
- note removed: "Flash"
- note removed: "PSRAM, 120MHz DDR OPI"
- note removed: "make sure not to get 8 instead of 9"
- moved on the sheet: C1, C10, C11, C13, C2, C21, C24, C25, C3, C30, C31, C4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

Commit message: nearly done with schematic i thinks
Parts:
- removed BT1: Battery, custom-lib:Battery_Connector, symbol Device:Battery
- removed C1, C10, C11, C2, C66, C67, C68, C69: C, symbol Device:C_Small
- removed C12, C19, C22: 22uF, symbol Device:C_Small
- removed C13, C21: 1.5pF, symbol Device:C_Small
- removed C14, C3, C44, C47, C50, C52, C53, C54, C55, C58, C61, C62, C64, C74, C75, C78, C79, C9: 100nF, symbol Device:C_Small
- removed C15, C33, C4, C48, C51, C56, C59, C6, C60, C63, C65, C72, C76: 1uF, symbol Device:C_Small
- removed C16, C20, C26, C27, C28, C29, C43, C5, C57, C7, C77, C80: 10uF, symbol Device:C_Small
- removed C17, C18, C49: 4.7uF, symbol Device:C_Small
- removed C23: 47nF, symbol Device:C_Small
- removed C37: 2.2uF, symbol Device:C_Small
- removed C70, C71: 1.5pF, Capacitor_SMD:C_0201_0603Metric, symbol Device:C_Small
- removed C73, C8: 10nF, symbol Device:C_Small
- removed D1: ESD9B5.0ST5G, Diode_SMD:D_SOD-923, symbol Diode:ESD9B5.0ST5G
- removed D2: CHARGING, symbol Device:LED
- removed D3: POWER GOOD, symbol Device:LED
- removed J1: USB_C_Receptacle, Connector_USB:USB_C_Receptacle_GCT_USB4105-xx-A_16P_TopMnt_Horizontal, symbol Connector:USB_C_Receptacle
- removed J2, J6: ESP_ANT, Connector_Coaxial:U.FL_Molex_MCRF_73412-0110_Vertical, symbol Connector:Conn_Coaxial_Small
- removed J4: Conn_01x06_Socket, symbol Connector:Conn_01x06_Socket
- removed J5: Micro_SD_Card, Connector_Card:microSD_HC_Hirose_DM3D-SF, symbol Connector:Micro_SD_Card
- removed JP6: RESET=LOW, Jumper:SolderJumper-2_P1.3mm_Open_RoundedPad1.0x1.5mm, symbol Jumper:SolderJumper_2_Open
- removed JP8: GP6, Jumper:SolderJumper-3_P1.3mm_Open_RoundedPad1.0x1.5mm, symbol Jumper:SolderJumper_3_Open
- removed L1: 1.5uH, symbol Device:L
- removed L2: 2.7nH, symbol Device:L
- removed L3, L4: 10uH, symbol Device:L
- removed L5: 1uH, symbol Device:L
- removed L7: 2.7nH, Inductor_SMD:L_0201_0603Metric, symbol Device:L
- removed L8: 2nH, symbol Device:L
- removed MK1: ICS-43434, Sensor_Audio:InvenSense_ICS-43434-6_3.5x2.65mm, symbol Sensor_Audio:ICS-43434
- removed R1, R2, R22: 5.1k, symbol Device:R
- removed R19, R20, R33, R34, R35, R36, R37, R38, R42, R43, R44, R45, R46, R47, R48, R49, R50, R51, R52, R53, R54: 10k, symbol Device:R
- removed R21: R, PCM_Resistor_SMD_AKL:R_0402_1005Metric, symbol Device:R
- removed R3: R, symbol Device:R
- removed R32: 100k, symbol Device:R
- removed R39: 5.24k, symbol Device:R
- removed R4: 180k, symbol Device:R
- removed R40: 30.31, symbol Device:R
- removed R5, R6: 1M, symbol Device:R
- removed R7: 1.5k, symbol Device:R
- removed SW1: USB, symbol Switch:SW_Push_Dual
- removed TH1: 103AT-2 10k, symbol Device:Thermistor_NTC
- removed TP2: FLASH RESET, symbol Connector:TestPoint
- removed TP3: RAM RESET, symbol Connector:TestPoint
- removed TP4: ECS, symbol Connector:TestPoint
- removed U1: DRV2605LYZFR, Package_BGA:Texas_DSBGA-9_1.4715x1.4715mm_Layout3x3_P0.5mm, symbol custom-lib:DRV2605LYZFR
- removed U10: APS12808L-3OBMx, custom-lib:BGA-24_6.0x8.0mm_Layout5x5_P1.0mm, symbol custom-lib:APS12808L-3OBMx
- removed U11: LSM6DSV16XTR, Package_LGA:LGA-14_3x2.5mm_P0.5mm_LayoutBorder3x4y, symbol custom-lib:LSM6DSV16XTR
- removed U12: ESP32-S3, Package_DFN_QFN:QFN-56-1EP_7x7mm_P0.4mm_EP4x4mm_ThermalVias, symbol MCU_Espressif:ESP32-S3
- removed U2: TPS63021, custom-lib:Texas_VSON-14_3x4mm_ThermalPad, symbol custom-lib:TPS63021
- removed U3: BQ25638, custom-lib:Texas_DSBGA-30_2.0x2.4mm_Layout5x6_P0.4mm, symbol custom-lib:BQ25638
- removed U4: TPS65631W, Package_SON:WSON-10-1EP_2.5x2.5mm_P0.5mm_EP1.2x2mm_ThermalVias, symbol custom-lib:TPS65631W
- removed U6: BQ27427YZFR, Package_BGA:Texas_DSBGA-9_1.4715x1.4715mm_Layout3x3_P0.5mm, symbol custom-lib:BQ27427YZFR
- removed U7: MAX30102, OptoDevice:Maxim_OLGA-14_3.3x5.6mm_P0.8mm, symbol Sensor:MAX30102
- removed U8: LIS3MDL, Package_LGA:LGA-12_2x2mm_P0.5mm, symbol Sensor_Magnetic:LIS3MDL
- removed U9: MX25LM51245GXDI00, custom-lib:BGA-24_6.0x8.0mm_Layout5x5_P1.0mm, symbol custom-lib:MX25LM51245GXDI00
- removed Y1, Y3: 40MHz(10ppm), Crystal:Crystal_SMD_3225-4Pin_3.2x2.5mm, symbol Device:Crystal_GND24_Small
- removed Y2, Y4: 32.768kHz, Crystal:Crystal_SMD_3215-2Pin_3.2x1.5mm, symbol Device:Crystal_Small
Connections:
- net I2C0_SCL: now also J3.4 (SCL)
- net I2C0_SDA: now also J3.3 (SDA)
- net I2C1_SCL: no longer J3.4 (SCL)
- net I2C1_SDA: no longer J3.3 (SDA)
- no-connect marks 15 -> 0
Other:
- added sheet IO (io.kicad_sch)
- added sheet MCU and Memory (mcu_mem.kicad_sch)
- added sheet USB and Power (usb_power.kicad_sch)
- note removed: "16MB PSRAM, 120MHz(133) DDR OPI"
- note removed: "1MHz"
- note removed: "400kHz"
- note removed: "64MB NOR Flash, 120MHz(133) DDR OPI"
- note removed: "CM315D32768HZFT"
- note removed: "FL4000157Z"
- note removed: "GOOD"
- note removed: "GRM0335C1H1R5BA01D"
- note removed: "LQP03TN2N7B02D"
- note removed: "gp44 gp43"
- note removed: "https://www.ti.com/lit/an/sloa207a/sloa207a.pdf?ts=1717055714895"
- note removed: "impedance match or something"
- note removed: "recalculate R for 0 1 imu"
- note removed: "std"

Commit message: basically done probably
Parts:
- removed C24, C30, C32, C35, C36, C45: 1uF, symbol Device:C_Small
- removed C25, C31, C34, C39, C40, C41, C42: 100nF, symbol Device:C_Small
- removed C38: 10nF, symbol Device:C_Small
- removed C46: 10uF, symbol Device:C_Small
- removed J3: TT143AMC12C, symbol custom-lib:TT143AMC12C
- removed JP2, JP3, JP4, JP5: GP6, Jumper:SolderJumper-3_P1.3mm_Open_RoundedPad1.0x1.5mm, symbol Jumper:SolderJumper_3_Open
- removed L6: 2nH, symbol Device:L
- removed R16, R17, R18: 0, symbol Device:R
- removed TP1: MTP_PWR, symbol Connector:TestPoint_Small
- removed U5: ESP32-S3, Package_DFN_QFN:QFN-56-1EP_7x7mm_P0.4mm_EP4x4mm_ThermalVias, symbol MCU_Espressif:ESP32-S3
- added D4: STATUS, symbol Device:LED
- added J4: DAUGHTER, symbol Connector:Conn_01x12_Pin
- added R1, R19: 10k, symbol Device:R
- R10, R11, R12, R13, R14, R15, R9: value 0 -> 10k
- R8: value 10k -> R
Connections:
- net +1V8: now also J4.2 (Pin_2)
- net +3V3: now also R10.2, R11.2, R12.2, R13.2, R14.2, R15.2, R9.2, J4.1 (Pin_1), R1.2, R19.2
- net GND: now also D4.1 (K), J4.12 (Pin_12)
- net MCU and Memory/EXT_IO11: now reaches R8.2
- net CPU_EN: no longer names the net of R8.1
- net CPU_EN: now also D4.2 (A)
- net MEM_CLK renamed IO/FI2C_SCL
- net MEM_D0 renamed SI2C_SDA
- net SI2C_SDA: now also J4.4 (Pin_4)
- net MEM_D1 renamed IO/IMU_SCL_PU
- net MEM_D2 renamed IO/FI2C_SDA
- net MEM_D3 renamed MCU and Memory/EXT_IO12
- net MEM_D4 renamed MCU and Memory/EXT_IO13
- net MEM_D5 renamed IO/HBT_INT
- new net IO/IMU_SDA_PU: R1.1
- new net MCU and Memory/EXT_IO10: J4.11 (Pin_11)
- new net MCU and Memory/EXT_IO6: J4.7 (Pin_7)
- new net MCU and Memory/EXT_IO7: J4.8 (Pin_8)
- new net MCU and Memory/EXT_IO8: J4.9 (Pin_9)
- new net MCU and Memory/EXT_IO9: J4.10 (Pin_10)
- new net MCU and Memory/IO7: J4.6 (Pin_6)
- new net PWR: J4.3 (Pin_3)
- new net SI2C_SCL: J4.5 (Pin_5), R19.1
Other:
- sheet IO ports: added DISP_CLK, DISP_CS, DISP_D0, DISP_D1, DISP_D2, DISP_D3, DISP_RST, DISP_TE, FI2C_SCL, FI2C_SDA, HBT_INT, IMU_INT1, IMU_INT2, IMU_SCL_PU, IMU_SDA_PU, MAG_DRDY, MAG_INT, MIC_SCK, MIC_SD, MIC_WS, MTR_EN, SI2C_SCL, SI2C_SDA, TP_INT, TP_RST; removed none
- sheet MCU and Memory ports: added BOOTSEL, EN, EXT_IO1, EXT_IO10, EXT_IO11, EXT_IO12, EXT_IO13, EXT_IO14, EXT_IO2, EXT_IO3, EXT_IO4, EXT_IO5, EXT_IO6, EXT_IO7, EXT_IO8, EXT_IO9, FSPI_CLK, FSPI_CS, FSPI_D, FSPI_HD, FSPI_Q, FSPI_WP, I2C0_SCL, I2C0_SDA, I2C1_SCL, I2C1_SDA, I2S_SCK, I2S_SD, I2S_WS, IO1, IO2, IO3, IO4, IO5, IO6, IO7, IO8, RX, TX; removed none
- sheet USB and Power ports: added 3V3_GOOD, 3V3_POWER_SAVE, BAT_LOW, BOOT, CHARGE_INT, MCU_RST, POWER_BTN, SCL, SDA, UART_RX, UART_TX; removed none
- note added: "1MHz"
- note added: "400kHz"
- note removed: "3v3=on"
