File: io.kicad_sch (KiCad schematic)
At the start: 39 parts, among them J2 MOTOR, J3 TT143AMC12C, U1 DRV2605LYZFR, U11 LSM6DSV16XTR, U4 TPS65631W, U7 MAX30102, U8 LIS3MDL

Commit message: switching to single repo
Other:
- note added: "0xD5 or 0xD7 2.6uA off 100uA normal 650uA highest performance"
Changed lines of the file:
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@@
+    (effects (font (size 1.27 1.27)) (justify left bottom))
+  )
+  (text "0xD5 or 0xD7\n2.6uA off\n100uA normal\n650uA highest performance"
+    (at 69.85 182.88 0)
     (effects (font (size 1.27 1.27)) (justify left bottom))
   )
