File: pcb/daughter-board/daughter-board.kicad_sch (KiCad schematic)
At the start: 16 parts, among them SW1 POWER, SW2 BTN1, SW3 BTN2, U1 VL53L1CXV0FY1

Commit message: finished pcb layout
Parts:
- removed SW1: POWER, symbol Switch:SW_Push
Changed lines of the file:
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@@
-    (stroke (width 0) (type default))
-  )
-  (wire (pts (xy 104.14 41.91) (xy 101.6 41.91))
     (stroke (width 0) (type default))
   )
@@
     (effects (font (size 1.27 1.27)) (justify right bottom))
   )
-  (label "POWER" (at 91.44 41.91 180) (fields_autoplaced)
-    (effects (font (size 1.27 1.27)) (justify right bottom))
-  )
   (label "SDA" (at 128.27 58.42 180) (fields_autoplaced)
     (effects (font (size 1.27 1.27)) (justify right bottom))
@@
         (path "/3fe54f5a-226a-46e4-ba63-4d629c108b01"
           (reference "D1") (unit 1)
-        )
-      )
-    )
-  )
-  (symbol (lib_id "Switch:SW_Push") (at 96.52 41.91 0) (unit 1)
-    (in_bom yes) (on_board yes) (dnp no) (fields_autoplaced)
-    (property "Reference" "SW1" (at 96.52 34.29 0)
-      (effects (font (size 1.27 1.27)))
-    )
-    (property "Value" "POWER" (at 96.52 36.83 0)
-      (effects (font (size 1.27 1.27)))
-    )
-    (property "Footprint" "" (at 96.52 36.83 0)
-      (effects (font (size 1.27 1.27)) hide)
-    )
-    (property "Datasheet" "~" (at 96.52 36.83 0)
-      (effects (font (size 1.27 1.27)) hide)
-    )
-    (pin "1")
-    (pin "2")
-    (instances
-      (project "daughter-board"
-        (path "/3fe54f5a-226a-46e4-ba63-4d629c108b01"
-          (reference "SW1") (unit 1)
         )
       )
@@
         )
       )
-    )
-  )
-  (symbol (lib_id "power:GND") (at 104.14 41.91 90) (unit 1)
-    (in_bom yes) (on_board yes) (dnp no) (fields_autoplaced)
-    (property "Reference" "#PWR06" (at 110.49 41.91 0)
-      (effects (font (size 1.27 1.27)) hide)
-    )
-    (property "Value" "GND" (at 107.95 41.91 90)
-      (effects (font (size 1.27 1.27)) (justify right))
-    )
-    (property "Footprint" "" (at 104.14 41.91 0)
-      (effects (font (size 1.27 1.27)) hide)
-    )
-    (property "Datasheet" "" (at 104.14 41.91 0)
-      (effects (font (size 1.27 1.27)) hide)
-    )
-    (pin "1")
-    (instances
-      (project "daughter-board"
-        (path "/3fe54f5a-226a-46e4-ba63-4d629c108b01"
-          (reference "#PWR06") (unit 1)
-        )
-      )
