File: pcb/io.kicad_sch (KiCad schematic)
At the start: 39 parts, among them J2 MOTOR, J3 TT143AMC12C, U1 DRV2605LYZFR, U11 LSM6DSV16XTR, U4 TPS65631W, U7 MAX30102, U8 LIS3MDL

Commit message: finished pcb layout
Parts:
- removed J2: MOTOR, custom-lib:Battery_Connector, symbol Connector_Generic:Conn_01x02
- added J5: ELV1411A, custom-lib:ELV1411A, symbol Connector:Conn_01x03_Pin
- C50: renamed from C14; footprint (none) -> Capacitor_SMD:C_0402_1005Metric
- C51: renamed from C3; footprint (none) -> Capacitor_SMD:C_0402_1005Metric
- C52: renamed from C20; footprint (none) -> Capacitor_SMD:C_0402_1005Metric
- C53: renamed from C4; footprint (none) -> Capacitor_SMD:C_0402_1005Metric
- C54: renamed from C10; footprint (none) -> Capacitor_SMD:C_0402_1005Metric
- C55: renamed from C11; footprint (none) -> Capacitor_SMD:C_0402_1005Metric
- C56: renamed from C6; footprint (none) -> Capacitor_SMD:C_0402_1005Metric
- C57: renamed from C13; footprint (none) -> Capacitor_SMD:C_0402_1005Metric
- C58: renamed from C21; footprint (none) -> Capacitor_SMD:C_0402_1005Metric
- C59: renamed from C49; footprint (none) -> Capacitor_SMD:C_0402_1005Metric
- C60: renamed from C50; footprint (none) -> Capacitor_SMD:C_0402_1005Metric
- C61: renamed from C51; footprint (none) -> Capacitor_SMD:C_0402_1005Metric
- C62: renamed from C26; footprint (none) -> Capacitor_SMD:C_0402_1005Metric
- C63: renamed from C28; footprint (none) -> Capacitor_SMD:C_0402_1005Metric
- C64: renamed from C24; footprint (none) -> Capacitor_SMD:C_0402_1005Metric
- C65: renamed from C25; footprint (none) -> Capacitor_SMD:C_0402_1005Metric
- C66: renamed from C30; footprint (none) -> Capacitor_SMD:C_0402_1005Metric
- C67: renamed from C31; footprint (none) -> Capacitor_SMD:C_0402_1005Metric
- C68: renamed from C32; footprint (none) -> Capacitor_SMD:C_0402_1005Metric
- C69: renamed from C34; footprint (none) -> Capacitor_SMD:C_0402_1005Metric
- C70: renamed from C33; footprint (none) -> Capacitor_SMD:C_0402_1005Metric
- C71: renamed from C37; footprint (none) -> Capacitor_SMD:C_0402_1005Metric
- C72: renamed from C43; footprint (none) -> Capacitor_SMD:C_0402_1005Metric
- C73: renamed from C44; footprint (none) -> Capacitor_SMD:C_0402_1005Metric
- C74: renamed from C47; footprint (none) -> Capacitor_SMD:C_0402_1005Metric
- C75: renamed from C48; footprint (none) -> Capacitor_SMD:C_0402_1005Metric
- J6: renamed from J3; footprint (none) -> custom-lib:OK-14GF024-04
- L7: renamed from L2; footprint (none) -> Inductor_SMD:L_1008_2520Metric
- L8: renamed from L3; footprint (none) -> Inductor_SMD:L_1008_2520Metric
- R54: renamed from R28; footprint (none) -> Resistor_SMD:R_0402_1005Metric
- TP1: footprint (none) -> TestPoint:TestPoint_Pad_D1.0mm
- renumbered MK2 to MK1, MK1 to MK2, U7 to U10, U4 to U11, U1 to U12, U11 to U13, U8 to U14
Connections:
- net GND: now also J6.25 (GND), J5.3 (Pin_3)
- net MTR_P: now reaches U12.A3 (OUT+)
- net MTR_P: now also J5.1 (Pin_1)
- net MTR_N: now reaches U12.C3 (OUT-)
- net MTR_N: now also J5.2 (Pin_2)
Other:
- moved on the sheet: C64, C65, C66, C67, TP1

Commit message: made many changes, maybe switching to stm tho
Parts:
- removed TP1: MTP_PWR, TestPoint:TestPoint_Pad_D1.0mm, symbol Connector:TestPoint_Small
Connections:
- net GND: now also J6.24 (MTP_PWR)
