File: pcb/usb_power.kicad_sch (KiCad schematic)
At the start: 59 parts, among them J7 USB_C_Receptacle, Q1 MBT2222ADW1T1, U14 CP2102N-Axx-xQFN28, U16 BQ25638, U17 ADP2108AUJ-1.8, U3 TPS63021, U5 BQ27427YZFR

Commit message: git is a tool for torture
Parts:
- removed Q1: MBT2222ADW1T1, Package_TO_SOT_SMD:SOT-363_SC-70-6, symbol Transistor_BJT:MBT2222ADW1T1
- removed R79: 1.5k, symbol Device:R
- added C38: 1uF, symbol Device:C_Small
- added Q1, Q2, Q3, Q4, Q5: MMBT3904, Package_TO_SOT_SMD:SOT-23, symbol Transistor_BJT:MMBT3904
- added R17: 6666, symbol Device:R
- added R18: 33k, symbol Device:R
- added R30: 2222, symbol Device:R
- C89: value 4.7uF -> 10uF
Connections:
- net DTR: now also Q1.2 (E)
- net GND: now also C38.2
- net ILIM: now also R17.1, R18.1, R30.1
- net RTS: now also Q5.2 (E)
- net at R65.1, R66.2, U14.8 (VBUS): now also C38.1
- net at R73.1: now also Q1.3 (C)
- net at R70.2: now also Q1.1 (B)
- net at R71.2: now also Q5.1 (B)
- net at R72.1: now also Q5.3 (C)
- net CH0: now reaches U14.13 (CHREN)
- net CH2: now reaches U14.14 (CHR1)
- net CH1: now reaches U14.15 (CHR0)

Commit message: finished pcb layout
Parts:
- added Q1: MMBT3904, Package_TO_SOT_SMD:SOT-23, symbol Transistor_BJT:MMBT3904
- C1: renamed from C15; footprint (none) -> Capacitor_SMD:C_0603_1608Metric
- C10: renamed from C98; footprint (none) -> Capacitor_SMD:C_0603_1608Metric
- C11: renamed from C1; footprint (none) -> Capacitor_SMD:C_0402_1005Metric
- C12: renamed from C88; footprint (none) -> Capacitor_SMD:C_0402_1005Metric
- C13: renamed from C89; footprint (none) -> Capacitor_SMD:C_0402_1005Metric
- C14: renamed from C5; footprint (none) -> Capacitor_SMD:C_0603_1608Metric
- C15: renamed from C2; footprint (none) -> Capacitor_SMD:C_0402_1005Metric
- C16: renamed from C7; footprint (none) -> Capacitor_SMD:C_0603_1608Metric
- C17: renamed from C8; footprint (none) -> Capacitor_SMD:C_0603_1608Metric
- C18: renamed from C90; footprint (none) -> Capacitor_SMD:C_0402_1005Metric
- C19: renamed from C91; footprint (none) -> Capacitor_SMD:C_0402_1005Metric
- C2: renamed from C16; footprint (none) -> Capacitor_SMD:C_0603_1608Metric
- C20: renamed from C92; footprint (none) -> Capacitor_SMD:C_0402_1005Metric
- C21: renamed from C93; footprint (none) -> Capacitor_SMD:C_0402_1005Metric
- C22: renamed from C94; footprint (none) -> Capacitor_SMD:C_0402_1005Metric
- C23: renamed from C95; footprint (none) -> Capacitor_SMD:C_0603_1608Metric
- C24: renamed from C96; footprint (none) -> Capacitor_SMD:C_0603_1608Metric
- C3: renamed from C23; footprint (none) -> Capacitor_SMD:C_0402_1005Metric
- C4: renamed from C17; footprint (none) -> Capacitor_SMD:C_0603_1608Metric
- C5: renamed from C18; footprint (none) -> Capacitor_SMD:C_0402_1005Metric
- C6: renamed from C97; footprint (none) -> Capacitor_SMD:C_0402_1005Metric
- C7: renamed from C27; footprint (none) -> Capacitor_SMD:C_0603_1608Metric
- C8: renamed from C29; footprint (none) -> Capacitor_SMD:C_0603_1608Metric
- C9: renamed from C38; footprint (none) -> Capacitor_SMD:C_0402_1005Metric
- D6: renamed from D5; footprint (none) -> LED_SMD:LED_0402_1005Metric
- D7: renamed from D8; footprint (none) -> LED_SMD:LED_0402_1005Metric
- L1: renamed from L5; footprint (none) -> custom-lib:XFL4020-152ME
- L2: renamed from L12; footprint (none) -> Inductor_SMD:L_1206_3216Metric
- L3: renamed from L11; footprint (none) -> Inductor_SMD:L_1206_3216Metric
- R11: renamed from R39; footprint (none) -> Resistor_SMD:R_0402_1005Metric
- R12: renamed from R40; footprint (none) -> Resistor_SMD:R_0402_1005Metric
- R13: renamed from R76; footprint (none) -> Resistor_SMD:R_0402_1005Metric
- R14: renamed from R77; footprint (none) -> Resistor_SMD:R_0402_1005Metric
- R15: renamed from R78; footprint (none) -> Resistor_SMD:R_0402_1005Metric
- R16: renamed from R65; footprint (none) -> Resistor_SMD:R_0402_1005Metric
- R17: renamed from R66; footprint (none) -> Resistor_SMD:R_0402_1005Metric
- R18: renamed from R67; footprint (none) -> Resistor_SMD:R_0402_1005Metric
- R19: renamed from R3; footprint (none) -> Resistor_SMD:R_0402_1005Metric
- R20: renamed from R68; footprint (none) -> Resistor_SMD:R_0402_1005Metric
- R21: renamed from R69; footprint (none) -> Resistor_SMD:R_0402_1005Metric
- R22: renamed from R74; footprint (none) -> Resistor_SMD:R_0402_1005Metric
- R23: renamed from R30; footprint (none) -> Resistor_SMD:R_0402_1005Metric
- R24: renamed from R70; footprint (none) -> Resistor_SMD:R_0402_1005Metric
- R25: renamed from R71; footprint (none) -> Resistor_SMD:R_0402_1005Metric
- R26: renamed from R75; footprint (none) -> Resistor_SMD:R_0402_1005Metric
- R27: renamed from R17; footprint (none) -> Resistor_SMD:R_0402_1005Metric
- R28: renamed from R72; footprint (none) -> Resistor_SMD:R_0402_1005Metric
- R29: renamed from R73; footprint (none) -> Resistor_SMD:R_0402_1005Metric
- R30: renamed from R18; footprint (none) -> Resistor_SMD:R_0402_1005Metric
- TH1: renamed from TH2; footprint (none) -> Resistor_THT:R_Axial_DIN0204_L3.6mm_D1.6mm_P2.54mm_Vertical
- renumbered BT2 to BT1, D9 to D4, D1 to D5, J7 to J2, Q3 to Q2, Q5 to Q3, Q1 to Q4, Q2 to Q5, Q4 to Q6, U17 to U1, U3 to U2, U14 to U3, U5 to U4, U16 to U5
Connections:
- net +3V3: no longer U4.C2 (SRX)
- net +VSW: now also U4.C2 (SRX)
- net CH0: now also Q6.1 (B)
- net CH1: now also Q5.1 (B)
- net CH2: now also Q2.1 (B)
- net GND: now also Q2.2 (E), Q5.2 (E), Q6.2 (E), Q1.2 (E); no longer C12.2, C13.1, U3.29 (GND), U3.3 (GND)
- net at Q2.3 (C): now also R23.2
- net at C9.1, R16.1, R17.2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: now also Q1.1 (B)
- net at Q6.3 (C): now also R30.2
- net at Q5.3 (C): now also R27.2
- new net: C12.2, C13.1, Q1.3 (C), U3.29 (GND), U3.3 (GND)
Other:
- note added: "LQM31PN1R0M00L"
- note added: "XFL4020-152ME"
- moved on the sheet: C3, C6, L2, Q2, Q5, Q6, R23, R27, R30, U1

Commit message: switching to 6 layer
Connections:
- net USB_DM renamed USB_DN
Changed lines of the file:
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@@
     (effects (font (size 1.27 1.27)) (justify right bottom))
   )
-  (label "USB_DM" (at 64.77 135.89 0) (fields_autoplaced)
+  (label "USB_DN" (at 64.77 135.89 0) (fields_autoplaced)
     (effects (font (size 1.27 1.27)) (justify left bottom))
   )
@@
     (effects (font (size 1.27 1.27)) (justify left bottom))
   )
-  (label "USB_DM" (at 110.49 149.86 180) (fields_autoplaced)
+  (label "USB_DN" (at 110.49 149.86 180) (fields_autoplaced)
     (effects (font (size 1.27 1.27)) (justify right bottom))
   )

Commit message: made many changes, maybe switching to stm tho
Parts:
- added R56, R57: R, Resistor_SMD:R_0402_1005Metric, symbol Device:R
- TH1: footprint Resistor_THT:R_Axial_DIN0204_L3.6mm_D1.6mm_P2.54mm_Vertical -> Resistor_SMD:R_0603_1608Metric
Connections:
- net +VSW: now also R56.2, R57.2; no longer D6.2 (A), D7.2 (A)
- new net: D7.2 (A), R56.1
- new net: D6.2 (A), R57.1
Other:
- moved on the sheet: D6, D7

Commit message: things
Parts:
- added C34, C37, C80, C81, C82, C83, C84, C85, C86: 100nF, symbol Device:C_Small
- added C87: 4.7uF, symbol Device:C_Small
- added U15: STM32H7S7A8I6, Package_BGA:UFBGA-169_7x7mm_Layout13x13_P0.5mm, symbol custom-lib:STM32H7S7A8I6
Connections:
- net +3V3: now also C34.1, C37.1, C80.1, C81.1, C82.1, C83.1, C84.1, C85.1, C86.1, C87.1, U15.C10 (VDD), U15.C3 (VDD), U15.C5 (VDD), U15.E11 (VDD), U15.G11 (VDD), U15.G3 (VDD), U15.K10 (VDD), U15.K2 (VDD), U15.L5 (VDD)
- net GND: now also C34.2, C37.2, C80.2, C81.2, C82.2, C83.2, C84.2, C85.2, C86.2, C87.2, U15.B9 (VSS), U15.C4 (VSS), U15.C6 (VSS), U15.C9 (VSS), U15.D11 (VSS), U15.F11 (VSS), U15.F3 (VSS), U15.F7 (VSS), U15.G6 (VSS), U15.G7 (VSS), U15.G8 (VSS), U15.H11 (VSS), U15.H7 (VSS), U15.J2 (VSS), U15.K11 (VSS), U15.L10 (VSS), U15.L6 (VSS), U15.L8 (VSS)
Other:
- moved on the sheet: C18, C19, C20, C21, C22, C23, C24, D6, D7, L3, Q2, Q5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

Commit message: what i said before
Parts:
- removed C12: 100nF, Capacitor_SMD:C_0402_1005Metric, symbol Device:C_Small
- removed C13, C19: 10uF, Capacitor_SMD:C_0402_1005Metric, symbol Device:C_Small
- removed C18, C9: 1uF, Capacitor_SMD:C_0402_1005Metric, symbol Device:C_Small
- removed C20, C21: 4.7uF, Capacitor_SMD:C_0402_1005Metric, symbol Device:C_Small
- removed C22: 47nF, Capacitor_SMD:C_0402_1005Metric, symbol Device:C_Small
- removed C23, C24: 10uF, Capacitor_SMD:C_0603_1608Metric, symbol Device:C_Small
- removed L3: 1uH, Inductor_SMD:L_1206_3216Metric, symbol Device:L
- removed Q1, Q2, Q3, Q4, Q5, Q6: MMBT3904, Package_TO_SOT_SMD:SOT-23, symbol Transistor_BJT:MMBT3904
- removed R16: 22.1k, Resistor_SMD:R_0402_1005Metric, symbol Device:R
- removed R17: 47.5k, Resistor_SMD:R_0402_1005Metric, symbol Device:R
- removed R18: 1k, Resistor_SMD:R_0402_1005Metric, symbol Device:R
- removed R20, R21, R28, R29: 0, Resistor_SMD:R_0402_1005Metric, symbol Device:R
- removed R22: 30.31, Resistor_SMD:R_0402_1005Metric, symbol Device:R
- removed R23: 2222, Resistor_SMD:R_0402_1005Metric, symbol Device:R
- removed R24, R25: 10k, Resistor_SMD:R_0402_1005Metric, symbol Device:R
- removed R26: 5.24k, Resistor_SMD:R_0402_1005Metric, symbol Device:R
- removed R27: 6666, Resistor_SMD:R_0402_1005Metric, symbol Device:R
- removed R30: 33k, Resistor_SMD:R_0402_1005Metric, symbol Device:R
- removed TH1: 103AT-2 10k, Resistor_SMD:R_0603_1608Metric, symbol Device:Thermistor_NTC
- removed U15: STM32H7S7A8I6, Package_BGA:UFBGA-169_7x7mm_Layout13x13_P0.5mm, symbol custom-lib:STM32H7S7A8I6
- removed U3: CP2102N-Axx-xQFN28, Package_DFN_QFN:QFN-28-1EP_5x5mm_P0.5mm_EP3.35x3.35mm, symbol Interface_USB:CP2102N-Axx-xQFN28
- removed U5: BQ25638, custom-lib:Texas_DSBGA-30_2.0x2.4mm_Layout5x6_P0.4mm, symbol custom-lib:BQ25638
- added C88: 4.7uF, Capacitor_SMD:C_0402_1005Metric, symbol Device:C_Small
- added C89, C90: 10uF, Capacitor_SMD:C_0402_1005Metric, symbol Device:C_Small
- added L4: 1uH, symbol Device:L
- added R60: 30.1, Resistor_SMD:R_0402_1005Metric, symbol Device:R
- added R61: 5.32k, Resistor_SMD:R_0402_1005Metric, symbol Device:R
- added R62: 5k, Resistor_SMD:R_0402_1005Metric, symbol Device:R
- added TH2: 103AT-2 10k, Resistor_SMD:R_0603_1608Metric, symbol Device:Thermistor_NTC
- added U3: STM32H7S7L8H6H, Package_BGA:ST_TFBGA-225_13x13mm_Layout15x15_P0.8mm, symbol custom-lib:STM32H7S7L8H6H
- added U6: BQ25628E, custom-lib:Texas_WQFN-18_2.5x3.0mm_P0.4mm, symbol custom-lib:BQ25628E
- C14: value 22uF -> 1uF; footprint Capacitor_SMD:C_0603_1608Metric -> Capacitor_SMD:C_0402_1005Metric
- C16: value 22uF -> 47nF; footprint Capacitor_SMD:C_0603_1608Metric -> Capacitor_SMD:C_0402_1005Metric
- C17: value 22uF -> 100nF; footprint Capacitor_SMD:C_0603_1608Metric -> Capacitor_SMD:C_0402_1005Metric
Connections:
- net +3V3: now also R56.2, R57.2
- net +BATT: now also C90.1, U6.8 (BAT); no longer C14.1, C16.1, C17.1
- net +VSW: now also L4.2, U6.9 (SYS); no longer R56.2, R57.2
- net CHARGE_INT: now also U6.11 (INT)
- net GND: now also C88.2, C89.1, C90.2, R60.1, R62.2, TH2.1, U3.F15 (VSS), U3.F6 (VSS), U3.G10 (VSS), U3.G12 (VSS), U3.G8 (VSS), U3.H11 (VSS), U3.H7 (VSS), U3.H8 (VSS), U3.H9 (VSS), U3.J1 (VSS), U3.J10 (VSS), U3.J12 (VSS), U3.J15 (VSS), U3.J8 (VSS), U3.K7 (VSS), U3.K9 (VSS), U6.14 (CE), U6.15 (GND); no longer C16.2
- net ILIM: now also R62.1, U6.4 (ILIM)
- net POWER_BTN: now also U6.7 (QON)
- net SCL: now also U6.13 (SCL)
- net SDA: now also U6.12 (SDA)
- net VBUS: now also C14.1, U6.18 (VBUS)
- net at D7.2 (A): now also R57.1; no longer R56.1
- net at D6.1 (K): now also U6.10 (STAT)
- net at D6.2 (A): now also R56.1; no longer R57.1
- net at D7.1 (K): now also U6.3 (PG)
- new net: R60.2, R61.1, TH2.2, U6.6 (TS)
- new net: R61.2, U6.5 (TS_BIAS)
- new net: C17.1, C89.2, U6.17 (PMID)
- new net: C16.1, U6.1 (BTST)
- new net: C16.2, L4.1, U6.16 (SW)
- new net: C88.1, U6.2 (REGN)
- no-connect marks 24 -> 12
Other:
- moved on the sheet: BT1, C11, C15, C34, C37, C80, C81, C82, C83, C84, C85, C86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
