File: pcb/mcu_mem.kicad_sch (KiCad schematic)
At the start: 59 parts, among them J1 ESP_ANT, J5 Micro_SD_Card, U10 APS12808L-3OBMx, U2 ESP32-S3, U6 TCA9535MRGER, U9 MX25LM51245GXDI00, Y5 40MHz(10ppm), Y6 32.768kHz

Commit message: git is a tool for torture
Parts:
- added R16: 10k, symbol Device:R
Connections:
- net +3V3: now also R16.2
- net EN: now also R16.1
Changed lines of the file:
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@@
   (junction (at 87.63 38.1) (diameter 0) (color 0 0 0 0)
+  )
+  (junction (at 26.67 91.44) (diameter 0) (color 0 0 0 0)
   )
   (junction (at 135.89 88.9) (diameter 0) (color 0 0 0 0)
@@
     (stroke (width 0) (type default))
   )
+  (wire (pts (xy 26.67 88.9) (xy 26.67 91.44))
+    (stroke (width 0) (type default))
+  )
   (wire (pts (xy 135.89 173.99) (xy 153.67 173.99))
     (stroke (width 0) (type default))
@@
   )
   (symbol (lib_id "power:GND") (at 36.83 85.09 180) (unit 1)
-    (in_bom yes) (on_board yes) (dnp no) (fields_autoplaced)
+    (in_bom yes) (on_board yes) (dnp no)
     (property "Reference" "#PWR015" (at 36.83 78.74 0)
       (effects (font (size 1.27 1.27)) hide)
     )
-    (property "Value" "GND" (at 36.83 80.01 0)
+    (property "Value" "GND" (at 36.83 81.28 0)
       (effects (font (size 1.27 1.27)))
     )
@@
     )
   )
+  (symbol (lib_id "power:+3V3") (at 26.67 81.28 0) (unit 1)
+    (in_bom yes) (on_board yes) (dnp no)
+    (property "Reference" "#PWR060" (at 26.67 85.09 0)
+      (effects (font (size 1.27 1.27)) hide)
+    )
+    (property "Value" "+3V3" (at 26.67 77.47 0)
+      (effects (font (size 1.27 1.27)))
+    )
+    (property "Footprint" "" (at 26.67 81.28 0)
+      (effects (font (size 1.27 1.27)) hide)
+    )
+    (property "Datasheet" "" (at 26.67 81.28 0)
+      (effects (font (size 1.27 1.27)) hide)
+    )
+    (pin "1")
+    (instances
+      (project "watch-pcb"
+        (path "/b7b86b03-b0df-4b4e-be1d-606605306dad/1b63e572-6cfa-40af-85d8-9bf18f565a95"
+          (reference "#PWR060") (unit 1)
+        )
+      )
+    )
+  )
   (symbol (lib_id "Device:C_Small") (at 107.95 78.74 180) (unit 1)
     (in_bom yes) (on_board yes) (dnp no) (fields_autoplaced)
@@
         )
       )
+    )
+  )
+  (symbol (lib_id "Device:R") (at 26.67 85.09 180) (unit 1)
+    (in_bom yes) (on_board yes) (dnp no)
+    (property "Reference" "R16" (at 22.86 83.82 0)
+      (effects (font (size 1.27 1.27)))
+    )
+    (property "Value" "10k" (at 22.86 86.36 0)
+      (effects (font (size 1.27 1.27)))
+    )
+    (property "Footprint" "" (at 28.448 85.09 90)
+      (effects (font (size 1.27 1.27)) hide)
+    )
+    (property "Datasheet" "~" (at 26.67 85.09 0)
+      (effects (font (size 1.27 1.27)) hide)
+    )
+    (pin "1")
+    (pin "2")
+    (instances
+      (project "watch-pcb"
+        (path "/b7b86b03-b0df-4b4e-be1d-606605306dad/1b63e572-6cfa-40af-85d8-9bf18f565a95"
+          (reference "R16") (unit 1)
+        )
+      )

Commit message: finished pcb layout
Parts:
- removed C57: 10uF, symbol Device:C_Small
- added C45: 10uF, Capacitor_SMD:C_0402_1005Metric, symbol Device:C_Small
- added C76, C77, C78, C79: 100nF, Capacitor_SMD:C_0402_1005Metric, symbol Device:C_Small
- added D10, D11, D12, D13, D14, D8, D9: ESD9B3.3ST5G, Diode_SMD:D_SOD-923, symbol Diode:ESD9B3.3ST5G
- C26: renamed from C19; footprint (none) -> Capacitor_SMD:C_0402_1005Metric
- C27: renamed from C22; footprint (none) -> Capacitor_SMD:C_0402_1005Metric
- C28: renamed from C81; footprint (none) -> Capacitor_SMD:C_0402_1005Metric
- C30: renamed from C55; footprint (none) -> Capacitor_SMD:C_0402_1005Metric
- C31: renamed from C56; footprint (none) -> Capacitor_SMD:C_0402_1005Metric
- C32: renamed from C82; footprint (none) -> Capacitor_SMD:C_0402_1005Metric
- C33: renamed from C83; footprint (none) -> Capacitor_SMD:C_0402_1005Metric
- C34: renamed from C84; footprint (none) -> Capacitor_SMD:C_0402_1005Metric
- C35: renamed from C85; footprint (none) -> Capacitor_SMD:C_0402_1005Metric
- C36: renamed from C86; footprint (none) -> Capacitor_SMD:C_0402_1005Metric
- C37: renamed from C87; footprint (none) -> Capacitor_SMD:C_0402_1005Metric
- C38: renamed from C99; footprint (none) -> Capacitor_SMD:C_0402_1005Metric
- C39: renamed from C101; footprint (none) -> Capacitor_SMD:C_0402_1005Metric
- C40: renamed from C103; footprint (none) -> Capacitor_SMD:C_0402_1005Metric
- C41: renamed from C9; footprint (none) -> Capacitor_SMD:C_0402_1005Metric
- C42: renamed from C12; footprint (none) -> Capacitor_SMD:C_0402_1005Metric
- C43: renamed from C104; footprint (none) -> Capacitor_SMD:C_0402_1005Metric
- C44: renamed from C105; footprint (none) -> Capacitor_SMD:C_0402_1005Metric
- C46: renamed from C58; footprint (none) -> Capacitor_SMD:C_0402_1005Metric
- C47: renamed from C59; footprint (none) -> Capacitor_SMD:C_0402_1005Metric
- C48: renamed from C35; footprint (none) -> Capacitor_SMD:C_0402_1005Metric
- C49: renamed from C36; footprint (none) -> Capacitor_SMD:C_0402_1005Metric
- L5: renamed from L9; footprint (none) -> Inductor_SMD:L_0805_2012Metric
- L6: renamed from L1; footprint (none) -> Inductor_SMD:L_Coilcraft_XFL2010
- R31: renamed from R16; footprint (none) -> Resistor_SMD:R_0402_1005Metric
- R32: renamed from R2; footprint (none) -> Resistor_SMD:R_0402_1005Metric
- R33: renamed from R4; footprint (none) -> Resistor_SMD:R_0402_1005Metric
- R34: renamed from R5; footprint (none) -> Resistor_SMD:R_0402_1005Metric
- R35: renamed from R6; footprint (none) -> Resistor_SMD:R_0402_1005Metric
- R36: renamed from R7; footprint (none) -> Resistor_SMD:R_0402_1005Metric
- R37: renamed from R55; footprint (none) -> Resistor_SMD:R_0402_1005Metric
- R38: renamed from R56; footprint (none) -> Resistor_SMD:R_0402_1005Metric
- R40: renamed from R26; footprint (none) -> Resistor_SMD:R_0402_1005Metric
- R41: renamed from R58; footprint (none) -> Resistor_SMD:R_0402_1005Metric
- R42: renamed from R59; footprint (none) -> Resistor_SMD:R_0402_1005Metric
- R43: renamed from R60; footprint (none) -> Resistor_SMD:R_0402_1005Metric
- R44: renamed from R61; footprint (none) -> Resistor_SMD:R_0402_1005Metric
- R45: renamed from R62; footprint (none) -> Resistor_SMD:R_0402_1005Metric
- R46: renamed from R20; footprint (none) -> Resistor_SMD:R_0402_1005Metric
- R47: renamed from R21; footprint (none) -> Resistor_SMD:R_0402_1005Metric
- R48: renamed from R22; footprint (none) -> Resistor_SMD:R_0402_1005Metric
- R49: renamed from R23; footprint (none) -> Resistor_SMD:R_0402_1005Metric
- R50: renamed from R24; footprint (none) -> Resistor_SMD:R_0402_1005Metric
- R51: renamed from R25; footprint (none) -> Resistor_SMD:R_0402_1005Metric
- R52: renamed from R27; footprint (none) -> Resistor_SMD:R_0402_1005Metric
- R53: renamed from R29; footprint (none) -> Resistor_SMD:R_0402_1005Metric
- renumbered C100 to C25, C102 to C29, J1 to J3, J5 to J4, JP7 to JP1, L13 to L4, R57 to R39, U2 to U6, U9 to U7, U10 to U8, U6 to U9, Y6 to Y1, Y5 to Y2
Connections:
- net +3V3: now also C45.2, C76.1, C77.1, C78.1, C79.1, D14.2 (A2)
- net GND: now also C38.2, C39.2, C40.2, C43.2, C44.2, C45.1, C76.2, C77.2, C78.2, C79.2, D10.1 (A1), D11.1 (A1), D12.1 (A1), D13.1 (A1), D14.1 (A1), D8.1 (A1), D9.1 (A1)
- net SD_CLK: now also D11.2 (A2)
- net SD_CMD: now also D10.2 (A2)
- net SD_D0: now also D12.2 (A2)
- net SD_D1: now also D13.2 (A2)
- net SD_D2: now also D8.2 (A2)
- net SD_D3: now also D9.2 (A2)
- no-connect marks 1 -> 0
Other:
- note removed: "std"
- moved on the sheet: C26, C30, C31, C32, C33, C34, C35, C36, C37, C38, C39, C40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

Commit message: made many changes, maybe switching to stm tho
Parts:
- removed C34: 1uF, Capacitor_SMD:C_0402_1005Metric, symbol Device:C_Small
- removed C37: 100nF, Capacitor_SMD:C_0402_1005Metric, symbol Device:C_Small
Connections:
- net +3V3: now also C32.2, C35.2, U6.20 (VDD3P3_RTC), U6.46 (VDD3P3_CPU)
- net SD_CLK: now also U6.48 (MTMS); no longer U6.36 (SPICLK_N)
- net SD_CMD: now also U6.47 (MTDI); no longer U6.37 (SPICLK_P)
- net SD_D0: now also U6.37 (SPICLK_P); no longer U6.44 (MTCK)
- net SD_D1: now also U6.36 (SPICLK_N); no longer U6.45 (MTDO)
- net SD_D2: now also U6.44 (MTCK); no longer U6.47 (MTDI)
- net SD_D3: now also U6.45 (MTDO); no longer U6.48 (MTMS)
- no-connect marks 0 -> 1

Commit message: things
Parts:
- removed C25, C29: 1.5pF, Capacitor_SMD:C_0201_0603Metric, symbol Device:C_Small
- removed J3: ESP_ANT, Connector_Coaxial:U.FL_Molex_MCRF_73412-0110_Vertical, symbol Connector:Conn_Coaxial_Small
- removed L4: 2.7nH, Inductor_SMD:L_0201_0603Metric, symbol Device:L
- removed U6: ESP32-S3, Package_DFN_QFN:QFN-56-1EP_7x7mm_P0.4mm_EP4x4mm_ThermalVias, symbol MCU_Espressif:ESP32-S3
Other:
- note removed: "GRM0335C1H1R5BA01D"
- note removed: "LQP03TN2N7B02D"

Commit message: returning and reorganizing
Parts:
- removed C45: 10uF, Capacitor_SMD:C_0402_1005Metric, symbol Device:C_Small
- removed D10, D11, D12, D13, D14, D8, D9: ESD9B3.3ST5G, Diode_SMD:D_SOD-923, symbol Diode:ESD9B3.3ST5G
- removed J4: Micro_SD_Card, Connector_Card:microSD_HC_Hirose_DM3D-SF, symbol Connector:Micro_SD_Card
- removed R46, R47, R48, R49, R50, R51: 10k, Resistor_SMD:R_0402_1005Metric, symbol Device:R
