File: pcb/stm_mcu.kicad_sch (KiCad schematic)
At the start: 15 parts, among them J3 Micro_SD_Card, U3 STM32H7S7L8H6H, U5 APS256XXN-OBR-BG, Y3 32.768kHz

Commit message: returning and reorganizing
Parts:
- removed R58, R59: 0, symbol Device:R
- added C100, C23, C24, C34, C37, C41, C42, C44, C47, C80, C81, C82, C85, C86, C87, C91, C93, C94, C95, C96, C97, C98: 100nF, symbol Device:C_Small
- added C101, C43, C46, C84, C92, C99: 1uF, symbol Device:C_Small
- added C103: 100n, symbol Device:C_Small
- added C21, C22: C, Capacitor_SMD:C_0402_1005Metric, symbol Device:C_Small
- added C45: 1uF, Capacitor_SMD:C_0402_1005Metric, symbol Device:C_Small
- added C48: 4.7u, symbol Device:C_Small
- added C77, C78, C79: 2.2u, symbol Device:C_Small
- added C83: 4.7uF, symbol Device:C_Small
- added D8, D9: ESD9B5.0ST5G, Diode_SMD:D_SOD-923, symbol Diode:ESD9B5.0ST5G
- added FB1, FB2, FB3: ~, symbol Device:FerriteBead_Small
- added J8: SWD, symbol Connector:Conn_01x03_Socket
- added JP1: CS12, Jumper:SolderJumper-3_P1.3mm_Open_RoundedPad1.0x1.5mm_NumberLabels, symbol Jumper:SolderJumper_3_Bridged12
- added R17, R18: 10k, symbol Device:R
- added R23, R24: 0, symbol Device:R
- added U15: TXS02612RTW, Package_DFN_QFN:WQFN-24-1EP_4x4mm_P0.5mm_EP2.45x2.45mm_ThermalVias, symbol Logic_LevelTranslator:TXS02612RTW
- added unit 2 of U3
- added Y4: 40MHz(10ppm), Crystal:Crystal_SMD_3225-4Pin_3.2x2.5mm, symbol Device:Crystal_GND24_Small
- J3: footprint (none) -> Connector_Card:microSD_HC_Molex_104031-0811
Connections:
- net +1V8: now also C19.1, C20.1, J3.4 (VDD), U3.C1 (VBAT), U3.L9 (VDD), C100.2, C101.2, C23.1, C24.1, C34.1, C37.1, C41.2, C42.1, C46.2, C47.2, C80.1, C81.1, C82.1, C83.1, C86.1, C87.1, C91.1, C92.1, C93.1, C94.1, C95.1, C96.1, C97.1, C98.1, C99.1, FB1.2, R17.1, U15.17 (VCC_{B1}), U15.21 (VCC_{B0}), U15.5 (V_{CCA}), U3.F10 (VDD), U3.F7 (VDD), U3.F9 (VDD), U3.G6 (VDD), U3.G7 (VDDLDO), U3.G9 (VDDLDO), U3.H10 (VDD), U3.H12 (VDDXSPI_2), U3.H6 (VDD), U3.J11 (VDDXSPI_2), U3.J7 (VDDLDO), U3.J9 (VDDLDO), U3.K10 (VDD), U3.K12 (VDDXSPI_2), U3.K5 (VREFP), U3.K6 (VDD), U3.K8 (VDD)
- net BOOT: now also R17.2, R18.1; no longer U3.A6 (BOOT0)
- net GND: now also C100.1, C101.1, C103.2, C21.2, C22.1, C23.2, C24.2, C34.2, C37.2, C41.1, C42.2, C43.2, C44.2, C45.2, C46.1, C47.1, C48.2, C77.2, C78.2, C79.2, C80.2, C81.2, C82.2, C83.2, C84.1, C85.1, C86.2, C87.2, C91.2, C92.2, C93.2, C94.2, C95.2, C96.2, C97.2, C98.2, C99.2, D8.1 (A1), D9.2 (A2), J8.2 (Pin_2), U15.11 (GND), U15.2 (GND), U15.24 (SEL), U15.25 (EPAD), U3.F15 (VSS), U3.F6 (VSS), U3.G10 (VSS), U3.G12 (VSS), U3.G2 (VFBSMP_S), U3.G8 (VSS), U3.H1 (VDDSMP_S), U3.H11 (VSS), U3.H2 (VSSSMP_S), U3.H7 (VSS), U3.H8 (VSS), U3.H9 (VSS), U3.J1 (VSS), U3.J10 (VSS), U3.J12 (VSS), U3.J15 (VSS), U3.J5 (VSSA), U3.J8 (VSS), U3.K4 (VREFM), U3.K7 (VSS), U3.K9 (VSS), Y4.2, Y4.4
- net RTC_CLK_P: now reaches U3.D2 (PC14-_OSC32_I_N)
- net RTC_CLK_P: now also R23.1
- net at C25.1, Y3.2: now also R23.2
- net at U3.L15 (PN12): now also JP1.1 (A)
- net VCAP: now reaches U3.L7 (VCAP1)
- net VCAP: now also U3.D8 (DVDD), U3.E6 (VCAP4), C103.1, C77.1, C78.1, C79.1, U3.F11 (VCAP3), U3.K11 (VCAP2)
- net I2S1_WS: now reaches U3.M3 (PA4)
- net I2S1_SCK: now reaches U3.N2 (PA5)
- net I2S1_SD: now reaches U3.P1 (PA6)
- net IO4: now reaches U3.A12 (PD3)
- net IO5: now reaches U3.A13 (PE14)
- net SD_HOST_CMD: now reaches U3.A14 (PD2)
- net SD_HOST_CMD: now also U15.4 (CMDA)
- net IO0: now reaches U3.A2 (PE0)
- net IO1: now reaches U3.A3 (PF3)
- net IO2: now reaches U3.A4 (PF2)
- net IO3: now reaches U3.A5 (PG3)
- net USB_DM: now reaches U3.A7 (PM12)
- net I2C1_SCL: now reaches U3.B1 (PB8)
- net IO10: now reaches U3.B11 (PG0)
- net IO11: now reaches U3.B12 (PE13)
- net IO12: now reaches U3.B13 (PD1)
- net SD_HOST_D2: now reaches U3.B14 (PC10)
- net SD_HOST_D2: now also U15.1 (DAT2A)
- net SD_HOST_D3: now reaches U3.B15 (PC11)
- net SD_HOST_D3: now also U15.3 (DAT3A)
- net IO6: now reaches U3.B2 (PE2)
- net IO7: now reaches U3.B3 (PB5)
- net IO8: now reaches U3.B4 (PF4)
- net I2C2_SDA: now reaches U3.B5 (PF0)
- net IO9: now reaches U3.B6 (PD7)
- net USB_DP: now reaches U3.B7 (PM11)
- net IO32: now reaches U3.C11 (PD4)
- net IO31: now reaches U3.C12 (PE11)
- net IO30: now reaches U3.C13 (PD0)
- net IO29: now reaches U3.C14 (PA12)
- net IO28: now reaches U3.C15 (PA11)
- net I2C1_SDA: now reaches U3.C2 (PB9)
- net IO13: now reaches U3.C3 (PE1)
- net IO14: now reaches U3.C4 (PB3)
- net I2C2_SCL: now reaches U3.C5 (PF1)
- net SYNC: now reaches U3.C6 (PG2)
- net +5V: now reaches U3.C8 (PM14)
- net RTC_CLK_M: now reaches U3.D1 (PC15-_OSC32_O_UT)
- net RTC_CLK_M: now also R24.1
- net IO24: now reaches U3.D11 (PE15)
- net SD_HOST_CLK: now reaches U3.D12 (PC12)
- net SD_HOST_CLK: now also U15.9 (CLKA)
- net SWCLK: now reaches U3.D13 (PA14)
- net SWCLK: now also D9.1 (A1), J8.3 (Pin_3)
- net I2C3_SDA: now reaches U3.D14 (PA9)
- net SD_HOST_D0: now reaches U3.D15 (PC8)
- net SD_HOST_D0: now also U15.6 (DAT0A)
- net IO27: now reaches U3.D4 (PB7)
- net IO26: now reaches U3.D5 (PB4)
- net IO25: now reaches U3.D7 (PD5)
- net +3V3: now reaches U3.D9 (VDD50US_B)
- net +3V3: now also C43.1, C44.1, C48.1, U3.F8 (VDD33US_B)
- net IO23: now reaches U3.E1 (PE6)
- net IO18: now reaches U3.E10 (PG1)
- net IO17: now reaches U3.E11 (PE12)
- net SWDIO: now reaches U3.E12 (PA13)
- net SWDIO: now also D8.2 (A2), J8.1 (Pin_1)
- net IO16: now reaches U3.E13 (PA10)
- net SD_HOST_D1: now reaches U3.E14 (PC9)
- net SD_HOST_D1: now also U15.7 (DAT1A)
- net IO22: now reaches U3.E2 (PE4)
- net RTC0: now reaches U3.E4 (PC13)
- net IO20: now reaches U3.E5 (PB6)
- net IO19: now reaches U3.E7 (PD6)
- net at C29.1, Y3.1: now also R24.2
- net SD_DEV_D2: now reaches J3.1 (DAT2)
- net SD_DEV_D2: now also U15.23 (DAT2_{B0})
- net SD_DEV_D3: now reaches J3.2 (DAT3/CD)
- net SD_DEV_D3: now also U15.22 (DAT3_{B0})
- net SD_DEV_CMD: now reaches J3.3 (CMD)
- net SD_DEV_CMD: now also U15.20 (CMD_{B0})
- net SD_DEV_CLK: now reaches J3.5 (CLK)
- net SD_DEV_CLK: now also U15.19 (CLK_{B0})
- net SD_DEV_D0: now reaches J3.7 (DAT0)
- net SD_DEV_D0: now also U15.18 (DAT0_{B0})
- net SD_DEV_D1: now reaches J3.8 (DAT1)
- net SD_DEV_D1: now also U15.16 (DAT1_{B0})
- new net: C45.1, R18.2, U3.A6 (BOOT0)
- new net: C84.2, C85.2, FB1.1, U3.J6 (VDDA)
- new net: C21.1, FB2.2, Y4.1
- new net: C22.2, FB3.2, Y4.3
- new net CLK_M: FB3.1, U3.K2 (PH1-_OSC_OU_T)
- new net CLK_P: FB2.1, U3.K1 (PH0-_OSC_IN)
- new net I2C3_SCL: U3.F12 (PA8)
- new net MCU_RST: U3.J4 (NRST)
- new net QSPI1_CS: JP1.3 (B), U3.F14 (PN1)
- new net QSPI1_D0: U3.H15 (PN2)
- new net QSPI1_D2: U3.K14 (PN4)
- new net QSPI1_D3: U3.K15 (PN5)
- new net QSPI2_CS: JP1.2 (C)
- new net QSPI2_D0: U3.K13 (PN8)
- new net QSPI2_D1: U3.H14 (PN9)
- new net QSPI2_D2: U3.H13 (PN10)
- new net QSPI2_D3: U3.G15 (PN11)
- new net QSPI_CLK: U3.J14 (PN6)
- new net QSPI_D1: U3.G13 (PN3)
- no-connect marks 0 -> 17
Other:
- note added: "ESP8685H4 eventually on daughter board"
- note added: "an2867 has clock guidelines"
- note added: "connect to another pin"
- note added: "stm says left methinks right"
- note removed: "stm32wb09te eventually on daughter board"
- moved on the sheet: C12, C13, C18, C19, C20, C9, J3, R16, U3A, U3C, U5
