File: pcb/watch-pcb.kicad_pcb (KiCad board)
At the start: 6 copper layers, 43 x 43 mm, 167 parts, among them IC1 APS256XXN-OBR-BG, J1 DAUGHTER, J2 USB_C_Receptacle, J4 Micro_SD_Card, J5 ELV1411A, J6 TT143AMC12C, U1 ADP2108AUJ-1.8, U10 MAX30102, U11 TPS65631W, U12 DRV2605LYZFR, U13 LSM6DSV16XTR, U14 LIS3MDL, U2 TPS63021, U3 STM32H7S7L8H6H, U4 BQ27427YZFR, U6 BQ25628E, U7 MX25LM51245GXDI00, U8 APS12808L-3OBMx, U9 TCA9535MRGER, Y1 32.768kHz, Y2 40MHz(10ppm), Y3 32.768kHz

Commit message: returning and reorganizing
Parts:
- removed C51: 100nF, Capacitor_SMD:C_0402_1005Metric
- removed C53, C56: 1uF, Capacitor_SMD:C_0402_1005Metric
- removed D10, D11, D12, D13, D14, D8, D9: ESD9B3.3ST5G, Diode_SMD:D_SOD-923
- removed IC1: APS256XXN-OBR-BG, custom-lib:BGA-24_6.0x8.0mm_Layout5x5_P1.0mm
- removed J5: ELV1411A, custom-lib:ELV1411A
- removed R46, R47, R48, R49, R50, R51: 10k, Resistor_SMD:R_0402_1005Metric
- removed U12: DRV2605LYZFR, Package_BGA:Texas_DSBGA-9_1.4715x1.4715mm_Layout3x3_P0.5mm
- added C104: 1uF, Capacitor_SMD:C_0402_1005Metric, F.Cu at (90.5, 38.8)
- added C105: 100nF, Capacitor_SMD:C_0402_1005Metric, F.Cu at (90.5, 40.8)
- added C106: 1uF, Capacitor_SMD:C_0402_1005Metric, F.Cu at (90.5, 42.7)
- added C21: C, Capacitor_SMD:C_0402_1005Metric, F.Cu at (169.4, 73.8)
- added C22: C, Capacitor_SMD:C_0402_1005Metric, F.Cu at (169.4, 75.8)
- added J3: Micro_SD_Card, Connector_Card:microSD_HC_Molex_104031-0811, F.Cu at (152.8, 27.9)
- added U15: TXS02612RTW, Package_DFN_QFN:WQFN-24-1EP_4x4mm_P0.5mm_EP2.45x2.45mm_ThermalVias, F.Cu at (140.2, 29.0)
- added U16: DRV2605LDGS, Package_SO:VSSOP-10_3x3mm_P0.5mm, F.Cu at (95.7, 40.1)
- added U5: APS256XXN-OBR-BG, custom-lib:BGA-24_6.0x8.0mm_Layout5x5_P1.0mm, B.Cu at (129.6, 39.2)
- added Y4: 40MHz(10ppm), Crystal:Crystal_SMD_3225-4Pin_3.2x2.5mm, F.Cu at (118.8, 36.8)
- C45: value 10uF -> 1uF
- J4: value Micro_SD_Card -> ELV1411A; footprint Connector_Card:microSD_HC_Hirose_DM3D-SF -> custom-lib:ELV1411A
- U4: footprint Package_BGA:Texas_DSBGA-9_1.4715x1.4715mm_Layout3x3_P0.5mm -> Package_BGA:Texas_DSBGA-9_1.62mmx1.58mm_Layout3x3_P0.5mm
- moved Y3 17.7 mm to (143.7, 38.2)
- moved U6 12.8 mm to (144.2, 53.1)
Connections:
- net /USB and Power/USB_DN renamed /USB and Power/USB_DM
- C45 pad 1: GND -> Net-(U3A-BOOT0)
- C45 pad 2: +3V3 -> GND
- J4 pad 1: /MCU and Memory/SD_D2 -> unconnected-(J4-Pin_1-Pad1)
- J4 pad 2: /MCU and Memory/SD_D3 -> unconnected-(J4-Pin_2-Pad2)
- J4 pad 3: /MCU and Memory/SD_CMD -> unconnected-(J4-Pin_3-Pad3)
- J6 pad 3: /SI2C_SDA -> /IO/SI2C_SDA
- J6 pad 4: /SI2C_SCL -> /IO/SI2C_SCL
- R10 pad 1: /IO/IMU_SCL -> /IMU_SCL_PU
- R4 pad 1: /SI2C_SDA -> unconnected-(R4-Pad1)
- R5 pad 1: /SI2C_SCL -> unconnected-(R5-Pad1)
- R6 pad 1: /IO/FI2C_SDA -> unconnected-(R6-Pad1)
- R7 pad 1: /IO/FI2C_SCL -> unconnected-(R7-Pad1)
- R8 pad 1: /IO/HBT_INT -> unconnected-(R8-Pad1)
- R9 pad 1: /IO/IMU_SDA -> /IMU_SDA_PU
- U13 pad 2: /IO/IMU_SDA -> unconnected-(U13-SDx/AH1/QVAR1-Pad2)
- U13 pad 3: /IO/IMU_SCL -> unconnected-(U13-SCx/AH2/QVAR2-Pad3)
- U3 pad A14: unconnected-(U3A-PD2-PadA14) -> /STM MCU/SD_HOST_CMD
- U3 pad A6: /STM MCU/BOOT -> Net-(U3A-BOOT0)
- U3 pad A9: unconnected-(U3A-PM6-PadA9) -> /STM MCU/USB_DP
- U3 pad B1: unconnected-(U3A-PB8-PadB1) -> /STM MCU/I2C1_SCL
- U3 pad B14: unconnected-(U3A-PC10-PadB14) -> /STM MCU/SD_HOST_D2
- U3 pad B15: unconnected-(U3A-PC11-PadB15) -> /STM MCU/SD_HOST_D3
- U3 pad B5: unconnected-(U3A-PF0-PadB5) -> /STM MCU/I2C2_SDA
- U3 pad B9: unconnected-(U3A-PM5-PadB9) -> /STM MCU/USB_DM
- U3 pad C1: unconnected-(U3A-VBAT-PadC1) -> +3V3
- U3 pad C2: unconnected-(U3A-PB9-PadC2) -> /STM MCU/I2C1_SDA
- U3 pad C5: unconnected-(U3A-PF1-PadC5) -> /STM MCU/I2C2_SCL
- U3 pad D1: Net-(U3A-PC15-_OSC32_O_UT) -> /STM MCU/RTC_CLK_M
- U3 pad D12: unconnected-(U3A-PC12-PadD12) -> /STM MCU/SD_HOST_CLK
- U3 pad D13: unconnected-(U3A-PA14-PadD13) -> /STM MCU/SWCLK
- U3 pad D14: unconnected-(U3A-PA9-PadD14) -> /STM MCU/I2C3_SDA
- U3 pad D15: unconnected-(U3A-PC8-PadD15) -> /STM MCU/SD_HOST_D0
- U3 pad D2: Net-(U3A-PC14-_OSC32_I_N) -> /STM MCU/RTC_CLK_P
- U3 pad E12: unconnected-(U3A-PA13-PadE12) -> /STM MCU/SWDIO
- U3 pad E14: unconnected-(U3A-PC9-PadE14) -> /STM MCU/SD_HOST_D1
- U3 pad F10: unconnected-(U3B-VDD-PadF10) -> +3V3
- U3 pad F12: unconnected-(U3B-PA8-PadF12) -> /STM MCU/I2C3_SCL
- U3 pad F14: unconnected-(U3B-PN1-PadF14) -> /STM MCU/QSPI_CS1
- U3 pad F7: unconnected-(U3B-VDD-PadF7) -> +3V3
- U3 pad F9: unconnected-(U3B-VDD-PadF9) -> +3V3
- U3 pad G13: unconnected-(U3B-PN3-PadG13) -> /STM MCU/QSPI_D1
- U3 pad G6: unconnected-(U3B-VDD-PadG6) -> +3V3
- U3 pad H10: unconnected-(U3B-VDD-PadH10) -> +3V3
- U3 pad H12: unconnected-(U3B-VDDXSPI_2-PadH12) -> +3V3
- U3 pad H15: unconnected-(U3B-PN2-PadH15) -> /STM MCU/QSPI_D0
- U3 pad H2: unconnected-(U3B-VSSSMP_S-PadH2) -> GND
- U3 pad H6: unconnected-(U3B-VDD-PadH6) -> +3V3
- U3 pad J11: unconnected-(U3B-VDDXSPI_2-PadJ11) -> +3V3
- U3 pad J14: unconnected-(U3B-PN6-PadJ14) -> /STM MCU/QSPI_CLK
- U3 pad J4: unconnected-(U3B-NRST-PadJ4) -> /STM MCU/MCU_RST
- U3 pad J5: unconnected-(U3B-VSSA-PadJ5) -> GND
- U3 pad J6: unconnected-(U3B-VDDA-PadJ6) -> Net-(U3B-VDDA)
- U3 pad K1: unconnected-(U3B-PH0-_OSC_IN-PadK1) -> /STM MCU/CLK_P
- U3 pad K10: unconnected-(U3B-VDD-PadK10) -> +3V3
- U3 pad K14: unconnected-(U3B-PN4-PadK14) -> /STM MCU/QSPI_D2
- U3 pad K15: unconnected-(U3B-PN5-PadK15) -> /STM MCU/QSPI_D3
- U3 pad K2: unconnected-(U3B-PH1-_OSC_OU_T-PadK2) -> /STM MCU/CLK_M
- U3 pad K6: unconnected-(U3B-VDD-PadK6) -> +3V3
- U3 pad K8: unconnected-(U3B-VDD-PadK8) -> +3V3
- U3 pad L9: unconnected-(U3C-VDD-PadL9) -> +3V3
- U3 pad M3: unconnected-(U3C-PA4-PadM3) -> /STM MCU/I2S1_WS
- U3 pad N2: unconnected-(U3C-PA5-PadN2) -> /STM MCU/I2S1_SCK
- U3 pad P1: unconnected-(U3C-PA6-PadP1) -> /STM MCU/I2S1_SD
- U9 pad 19: /SI2C_SDA -> /MCU and Memory/I2C0_SDA
- U9 pad 20: /SI2C_SCL -> /MCU and Memory/I2C0_SCL
- U9 pad 3: /IO/MAG_DRDY -> /MCU and Memory/EXT_IO1
- U9 pad 4: /IO/DISP_RST -> /MCU and Memory/EXT_IO2
- U9 pad 5: /IO/MTR_EN -> /MCU and Memory/EXT_IO3
- U9 pad 6: /IO/MAG_INT -> /MCU and Memory/EXT_IO4
- U9 pad 8: /IO/IMU_INT2 -> /MCU and Memory/EXT_IO6
- Y3 pad 1: Net-(C29-Pad1) -> /STM MCU/RTC_CLK_M
- Y3 pad 2: Net-(C25-Pad1) -> /STM MCU/RTC_CLK_P
Routing:
- net unconnected-(J4-Pin_3-Pad3): track 0.00 -> 158.2 mm, vias 0 -> 13
- net (no net): track 59.8 -> 124.2 mm, vias 14 -> 22
- net /MCU and Memory/SD_CMD: track 33.9 -> 0.00 mm, vias 3 -> 0
- net /MCU and Memory/SD_D2: track 33.3 -> 0.00 mm, vias 3 -> 0
- net /MCU and Memory/SD_D3: track 33.5 -> 0.87 mm, vias 3 -> 1
- net /MCU and Memory/SD_D0: track 29.4 -> 0.00 mm, vias 2 -> 0
- net /MCU and Memory/SD_D1: track 29.0 -> 0.00 mm, vias 3 -> 0
- net /USB and Power/CH0: track 15.3 -> 0.00 mm, vias 2 -> 0
- net unconnected-(U3A-PC8-PadD15): track 14.6 -> 0.00 mm, vias 2 -> 0
- net /USB and Power/CH2: track 11.2 -> 0.00 mm, vias 2 -> 0
- net /USB and Power/CH1: track 8.70 -> 0.00 mm, vias 2 -> 0
- net /USB and Power/RTS: track 6.02 -> 0.00 mm
- net /USB and Power/DTR: track 2.88 -> 0.00 mm
- net unconnected-(U3A-PM13-PadC7): track 0.00 -> 1.85 mm, vias 0 -> 1
- net Net-(U12-REG): track 1.78 -> 0.00 mm
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