File: pcb/watch-pcb.kicad_sch (KiCad schematic)
At the start: 12 parts, among them J4 DAUGHTER

Commit message: finished pcb layout
Parts:
- removed J4: DAUGHTER, symbol Connector:Conn_01x12_Pin
- added D15: STATUS0, LED_SMD:LED_0402_1005Metric, symbol Device:LED
- added J1: DAUGHTER, Connector_FFC-FPC:TE_1-1734839-2_1x12-1MP_P0.5mm_Horizontal, symbol Connector:Conn_01x12_Pin
- added R55: R, Resistor_SMD:R_0402_1005Metric, symbol Device:R
- D1: renamed from D4; value STATUS -> STATUS1; footprint (none) -> LED_SMD:LED_0402_1005Metric
- R1: renamed from R9; footprint (none) -> Resistor_SMD:R_0402_1005Metric
- R10: renamed from R12; footprint (none) -> Resistor_SMD:R_0402_1005Metric
- R2: renamed from R14; footprint (none) -> Resistor_SMD:R_0402_1005Metric
- R3: renamed from R8; footprint (none) -> Resistor_SMD:R_0402_1005Metric
- R4: renamed from R13; footprint (none) -> Resistor_SMD:R_0402_1005Metric
- R5: renamed from R19; footprint (none) -> Resistor_SMD:R_0402_1005Metric
- R6: renamed from R10; footprint (none) -> Resistor_SMD:R_0402_1005Metric
- R7: renamed from R11; footprint (none) -> Resistor_SMD:R_0402_1005Metric
- R8: renamed from R15; footprint (none) -> Resistor_SMD:R_0402_1005Metric
- R9: renamed from R1; footprint (none) -> Resistor_SMD:R_0402_1005Metric
Connections:
- net +1V8: now also J1.3 (Pin_3)
- net +3V3: now also J1.1 (Pin_1), J1.2 (Pin_2)
- net GND: now also D15.1 (K), J1.11 (Pin_11), J1.12 (Pin_12)
- net MCU and Memory/EXT_IO10: now also R55.2
- net MCU and Memory/EXT_IO7: now also J1.8 (Pin_8)
- net MCU and Memory/EXT_IO8: now also J1.9 (Pin_9)
- net MCU and Memory/EXT_IO9: now also J1.10 (Pin_10)
- net MCU and Memory/IO7: now also J1.7 (Pin_7)
- net SI2C_SCL: now also J1.5 (Pin_5)
- net SI2C_SDA: now also J1.4 (Pin_4)
- new net: D15.2 (A), R55.1
- new net MCU and Memory/IO6: J1.6 (Pin_6)
Other:
- moved on the sheet: D1, R3

Commit message: things
Other:
- added sheet STM MCU (stm_mcu.kicad_sch)
Changed lines of the file:
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@@
+	)
+	(sheet
+		(at 27.94 171.45)
+		(size 40.64 22.86)
+		(fields_autoplaced yes)
+		(stroke
+			(width 0.1524)
+			(type solid)
+		)
+		(fill
+			(color 0 0 0 0.0000)
+		)
+		(property "Sheetname" "STM MCU"
+			(at 27.94 170.7384 0)
+			(effects
+				(font
+					(size 1.27 1.27)
+				)
+				(justify left bottom)
+			)
+		)
+		(property "Sheetfile" "stm_mcu.kicad_sch"
+			(at 27.94 194.8946 0)
+			(effects
+				(font
+					(size 1.27 1.27)
+				)
+				(justify left top)
+			)
+		)
+		(instances
+			(project "watch-pcb"
+				(path "/b7b86b03-b0df-4b4e-be1d-606605306dad"
+					(page "5")
+				)
+			)
+		)
 	)
 	(sheet

Commit message: returning and reorganizing
Parts:
- removed R10, R9: 10k, Resistor_SMD:R_0402_1005Metric, symbol Device:R
Connections:
- net IO/HBT_INT: no longer R8.1
- net SI2C_SCL: no longer R5.1
- net SI2C_SDA: no longer R4.1
- net IO/FI2C_SCL: no longer names the net of R7.1
- net IO/FI2C_SDA: no longer names the net of R6.1
- net MCU and Memory/EXT_IO10: no longer names the net of R55.2
- net MCU and Memory/EXT_IO11: no longer names the net of R3.2
- net MCU and Memory/EXT_IO12 renamed USB and Power/BAT_LOW
- net MCU and Memory/EXT_IO13 renamed USB and Power/CHARGE_INT
- net MCU and Memory/EXT_IO7: no longer names the net of J1.8 (Pin_8)
- net MCU and Memory/EXT_IO8: no longer names the net of J1.9 (Pin_9)
- net MCU and Memory/EXT_IO9: no longer names the net of J1.10 (Pin_10)
- net MCU and Memory/IO6: no longer names the net of J1.6 (Pin_6)
- net MCU and Memory/IO7: no longer names the net of J1.7 (Pin_7)
Other:
- removed sheet MCU and Memory
- sheet IO ports: added ALT_DRDY, LASER, SCL1, SCL2, SCL3, SDA1, SDA2, SDA3, TP_COM_EN; removed FI2C_SCL, FI2C_SDA, IMU_SCL_PU, IMU_SDA_PU, SI2C_SCL, SI2C_SDA
- sheet STM MCU ports: added BOOT, I2C1_SCL, I2C1_SDA, I2C2_SCL, I2C2_SDA, I2C3_SCL, I2C3_SDA, I2S1_SCK, I2S1_SD, I2S1_WS, IO0, IO1, IO10, IO11, IO12, IO13, IO14, IO16, IO17, IO18, IO19, IO2, IO20, IO22, IO23, IO24, IO25, IO26, IO27, IO28, IO29, IO3, IO30, IO31, IO32, IO4, IO5, IO6, IO7, IO8, IO9, MCU_RST, QSPI1_CS, QSPI1_D0, QSPI1_D2, QSPI1_D3, QSPI2_CS, QSPI2_D0, QSPI2_D1, QSPI2_D2, QSPI2_D3, QSPI_CLK, QSPI_D1, RTC0, SYNC, USB_DM, USB_DP; removed none
- moved on the sheet: R4, R5, R6, R7, R8
